Commit message: Prety in RVIZ, a rock in Gazebo.

File: riptide_description/urdf/riptide.urdf (robot description, URDF)
Before this commit: robot riptide, 12 links, 11 joints
Links:
- removed link frame_link
- added link acoustics_link, mass 0.97; collision mesh filename=package://riptide_description/meshes/riptide_acoustics.stl; visual mesh filename=package://riptide_description/meshes/riptide_acoustics.stl
- added link chassis_link, mass 2.71; collision mesh filename=package://riptide_description/meshes/riptide_chassis.stl; visual mesh filename=package://riptide_description/meshes/riptide_chassis.stl
- added link housing_link, mass 9.59; collision mesh filename=package://riptide_description/meshes/riptide_housing.stl; visual mesh filename=package://riptide_description/meshes/riptide_housing.stl
- added link pneumatics_link, mass 1.3503; collision mesh filename=package://riptide_description/meshes/riptide_pneumatics.stl; visual mesh filename=package://riptide_description/meshes/riptide_pneumatics.stl
- added link port_battery_link, mass 1.867; collision mesh filename=package://riptide_description/meshes/riptide_port_battery.s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; visual mesh filename=package://riptide_description/meshes/riptide_port_battery.s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
- added link stbd_battery_link, mass 1.867; collision mesh filename=package://riptide_description/meshes/riptide_stbd_battery.s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; visual mesh filename=package://riptide_description/meshes/riptide_stbd_battery.s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
- link base_link: mass 48.84278656 -> None; geometry 
- link heave_port_aft_thruster: geometry collision cylinder length=0.1127 radius=0.0483; visual mesh filename=package://riptide_description/meshes/blue_robotics_t200.stl
- link heave_port_fwd_thruster: geometry collision cylinder length=0.1127 radius=0.0483; visual mesh filename=package://riptide_description/meshes/blue_robotics_t200.stl
- link heave_stbd_aft_thruster: geometry collision cylinder length=0.1127 radius=0.0483; visual mesh filename=package://riptide_description/meshes/blue_robotics_t200.stl
- link heave_stbd_fwd_thruster: geometry collision cylinder length=0.1127 radius=0.0483; visual mesh filename=package://riptide_description/meshes/blue_robotics_t200.stl
- link surge_port_hi_thruster: geometry collision cylinder length=0.1127 radius=0.0483; visual mesh filename=package://riptide_description/meshes/blue_robotics_t200.stl
- link surge_port_lo_thruster: geometry collision cylinder length=0.1127 radius=0.0483; visual mesh filename=package://riptide_description/meshes/blue_robotics_t200.stl
- link surge_stbd_hi_thruster: geometry collision cylinder length=0.1127 radius=0.0483; visual mesh filename=package://riptide_description/meshes/blue_robotics_t200.stl
- link surge_stbd_lo_thruster: geometry collision cylinder length=0.1127 radius=0.0483; visual mesh filename=package://riptide_description/meshes/blue_robotics_t200.stl
- link sway_aft_thruster: geometry collision cylinder length=0.1127 radius=0.0483; visual mesh filename=package://riptide_description/meshes/blue_robotics_t200.stl
- link sway_fwd_thruster: geometry collision cylinder length=0.1127 radius=0.0483; visual mesh filename=package://riptide_description/meshes/blue_robotics_t200.stl
Joints:
- removed joint base_frame
- added joint base_housing: type fixed, parent base_link, child housing_link, origin xyz=0.0737 0.0005 0.0621 rpy=0 0 0
- added joint chassis_acoustics: type fixed, parent chassis_link, child acoustics_link, origin xyz=0.1699 0 -0.0584 rpy=0 0 0
- added joint chassis_pneumatics: type fixed, parent chassis_link, child pneumatics_link, origin xyz=-0.1172 0 -0.0584 rpy=0 0 0
- added joint chassis_port_battery: type fixed, parent chassis_link, child port_battery_link, origin xyz=-0.1781 0.1302 -0.014 rpy=0 0 0
- added joint chassis_stbd_battery: type fixed, parent chassis_link, child stbd_battery_link, origin xyz=-0.1781 -0.1302 -0.014 rpy=0 0 0
- added joint housing_chassis: type fixed, parent housing_link, child chassis_link, origin xyz=-0.0556 0 -0.0749 rpy=0 0 0
- joint heave_port_aft_thruster_joint: origin xyz=-0.2724 0.1823 0.0077 rpy=0 0 0 -> xyz=-0.2724 0.1824 -0.0033 rpy=0 0 3.14159266; parent frame_link -> chassis_link
- joint heave_port_fwd_thruster_joint: origin xyz=0.2824 0.1823 0.007 rpy=0 0 0 -> xyz=0.2824 0.1824 -0.0033 rpy=0 0 3.14159266; parent frame_link -> chassis_link
- joint heave_stbd_aft_thruster_joint: origin xyz=-0.2724 -0.1823 0.0077 rpy=0 0 0 -> xyz=-0.2724 -0.1824 -0.0033 rpy=0 0 0; parent frame_link -> chassis_link
- joint heave_stbd_fwd_thruster_joint: origin xyz=0.2824 -0.1823 0.007 rpy=0 0 0 -> xyz=0.2824 -0.1824 -0.0033 rpy=0 0 0; parent frame_link -> chassis_link
- joint surge_port_hi_thruster_joint: origin xyz=-0.2128 0.1823 0.1384 rpy=0 0 0 -> xyz=-0.2238 0.1824 0.1384 rpy=0 -1.57079633 3.14159266; parent frame_link -> chassis_link
- joint surge_port_lo_thruster_joint: origin xyz=-0.2128 0.1823 -0.0762 rpy=0 0 0 -> xyz=-0.2238 0.1824 -0.0838 rpy=0 -1.57079633 3.14159266; parent frame_link -> chassis_link
- joint surge_stbd_hi_thruster_joint: origin xyz=-0.2128 -0.1823 0.1384 rpy=0 0 0 -> xyz=-0.2238 -0.1824 0.1384 rpy=0 1.57079633 0; parent frame_link -> chassis_link
- joint surge_stbd_lo_thruster_joint: origin xyz=-0.2128 -0.1823 -0.0762 rpy=0 0 0 -> xyz=-0.2238 -0.1824 -0.0838 rpy=0 1.57079633 0; parent frame_link -> chassis_link
- joint sway_aft_thruster_joint: origin xyz=-0.3744 0.0110 -0.0838 rpy=0 0 0 -> xyz=-0.3744 0.0000 -0.0838 rpy=0 -1.57079633 -1.57079633; parent frame_link -> chassis_link
- joint sway_fwd_thruster_joint: origin xyz=0.3776 0.0110 -0.0838 rpy=0 0 0 -> xyz=0.3776 0.0000 -0.0838 rpy=0 1.57079633 1.57079633; parent frame_link -> chassis_link

File: riptide_description/urdf/riptide.urdf.xacro (robot description, xacro)
@@ -7,111 +7,13 @@
 <!--                                  -->
 <robot name="riptide" xmlns:xacro="http://ros.org/wiki/xacro">
-  <xacro:property name="M_PI" value="3.14159266"/>
-  <xacro:include filename="t200_thrusters.urdf.xacro"/>
-  <link name="base_link">
-    <inertial>
-      <origin xyz="0.00043180 0.03202940 -0.13947140" rpy="0 0 0"/>
-      <mass value="34.47940950"/>
-      <inertia ixx="0.50862680" ixy="-0.00114566" ixz="-0.03874012"
-               iyy="1.70892348" iyz="-0.00286748"
-               izz="1.77586420"/>
-    </inertial>
-  </link>
-  <joint name="base_housing" type="fixed">
-    <origin xyz="0 0 0" rpy="0 0 0"/>
-    <parent link="base_link"/>
-    <child link="housing_link"/>
-  </joint>
-  <link name="housing_link">
-    <visual>
-      <origin xyz="0 0 0" rpy="0 0 0"/>
-      <geometry>
-        <mesh filename="package://riptide_description/meshes/riptide_housing.stl"/>
-      </geometry>
-      <material name="housing"/>
-    </visual>
-  </link>
-  <joint name="housing_chassis" type="fixed">
-    <origin xyz="-0.0556 0 -0.0749" rpy="0 0 0"/>
-    <parent link="housing_link"/>
-    <child link="chassis_link"/>
-  </joint>
-  <link name="chassis_link">
-    <visual>
-      <origin xyz="0 0 0" rpy="0 0 0"/>
-      <geometry>
-        <mesh filename="package://riptide_description/meshes/riptide_chassis.stl"/>
-      </geometry>
-      <material name="chassis"/>
-    </visual>
-  </link>
-  <joint name="chassis_acoustics" type="fixed">
-    <origin xyz="0.1699 0 -0.0584" rpy="0 0 0"/>
-    <parent link="chassis_link"/>
-    <child link="acoustic_link"/>
-  </joint>
-  <link name="acoustic_link">
-    <visual>
-      <origin xyz="0 0 0" rpy="0 0 0"/>
-      <geometry>
-        <mesh filename="package://riptide_description/meshes/riptide_acoustics.stl"/>
-      </geometry>
-      <material name="housing"/>
-    </visual>
-  </link>
-  <joint name="chassis_pneumatics" type="fixed">
-    <origin xyz="-0.1172 0 -0.0584" rpy="0 0 0"/>
-    <parent link="chassis_link"/>
-    <child link="pneumatic_link"/>
-  </joint>
-  <link name="pneumatic_link">
-    <visual>
-      <origin xyz="0 0 0" rpy="0 0 0"/>
-      <geometry>
-        <mesh filename="package://riptide_description/meshes/riptide_pneumatics.stl"/>
-      </geometry>
-      <material name="housing"/>
-    </visual>
-  </link>
-  <joint name="chassis_bat_port" type="fixed">
-    <origin xyz="-0.1781 0.1302 -0.0140" rpy="0 0 0"/>
-    <parent link="chassis_link"/>
-    <child link="bat_port_link"/>
-  </joint>
-  <link name="bat_port_link">
-    <visual>
-      <origin xyz="0 0 0" rpy="0 0 0"/>
-      <geometry>
-        <mesh filename="package://riptide_description/meshes/riptide_port_battery.stl"/>
-      </geometry>
-      <material name="housing"/>
-    </visual>
-  </link>
-  <joint name="chassis_bat_stbd" type="fixed">
-    <origin xyz="-0.1781 -0.1302 -0.0140" rpy="0 0 0"/>
-    <parent link="chassis_link"/>
-    <child link="bat_stbd_link"/>
-  </joint>
-  <link name="bat_stbd_link">
-    <visual>
-      <origin xyz="0 0 0" rpy="0 0 0"/>
-      <geometry>
-        <mesh filename="package://riptide_description/meshes/riptide_stbd_battery.stl"/>
-      </geometry>
-      <material name="housing"/>
-    </visual>
-  </link>
-  <joint name="base_imu" type="fixed">
-    <origin xyz="0 0 0" rpy="${M_PI} 0 0"/>
-    <parent link="base_link"/>
-    <child link="imu"/>
-  </joint>
-  <link name="imu">
-  </link>
+  <xacro:include filename="riptide_properties.urdf.xacro" />
+  <xacro:include filename="riptide_links.urdf.xacro" />
+  <xacro:include filename="riptide_joints.urdf.xacro" />
+  <xacro:include filename="t200_thrusters.urdf.xacro" />
   <material name="chassis">
-  <color rgba="0 0 0 1.0"/>
+    <color rgba="0 0 0 1.0"/>
   </material>
   <material name="housing">
-  <color rgba="0.2 0.2 0.2 1.0"/>
+    <color rgba="0.2 0.2 0.2 1.0"/>
   </material>
   <material name="thruster">

File: riptide_description/urdf/riptide_properties.urdf.xacro (robot description, xacro)
@@ -2,17 +2,53 @@
 <robot xmlns:xacro="http://ros.org/wiki/xacro">
   <xacro:property name="M_PI" value="3.14159266"/>
-  <xacro:property name="pitch_fix">
-    <origin xyz="0 0 0" rpy="0 ${M_PI/2} 0"/>
-  </xacro:property>
-  <xacro:property name="roll_fix">
-    <origin xyz="0 0 0" rpy="${M_PI/2} 0 0"/>
-  </xacro:property>
-  <xacro:property name="" value=""/>
-  <xacro:property name="_inertia">
-    <inertia ixx="" ixy="" ixz=""
-             iyy="" iyz=""
-             izz=""/>
-  </xacro:property>
-  <xacro:property name="_origin">
-    <origin xyz="" rpy=""/>
-  </xacro:property>
+  <xacro:property name="housing_camera_port" value="0.2744 0.04 -0.0004" />
+  <xacro:property name="housing_camera_stbd" value="0.2744 -0.04 -0.0004" />
+  <xacro:property name="housing_camera_down" value="0.236 0 -0.062" />
+  <xacro:property name="housing_depth_sensor" value="0 0 0.1049" />
+  <xacro:property name="housing_imu_one" value="0.1322 -0.0056 0.0268" />
+  <xacro:property name="housing_imu_two" value="-0.1469 0.0004 -0.0405" />
+  <xacro:property name="base_housing" value="0.0737 0.0005 0.0621" />
+  <xacro:property name="housing_chassis" value="-0.0556 0 -0.0749" />
+  <xacro:property name="chassis_acoustics" value="0.1699 0 -0.0584" />
+  <xacro:property name="chassis_pneumatics" value="-0.1172 0 -0.0584" />
+  <xacro:property name="chassis_port_battery" value="-0.1781 0.1302 -0.014" />
+  <xacro:property name="chassis_stbd_battery" value="-0.1781 -0.1302 -0.014" />
+  <xacro:property name="chassis_surge_port_hi" value="-0.2238 0.1824 0.1384" />
+  <xacro:property name="chassis_surge_port_lo" value="-0.2238 -0.1824 0.1384" />
+  <xacro:property name="chassis_surge_port_lo" value="-0.2238 0.1824 -0.0838" />
+  <xacro:property name="chassis_surge_stbd_lo" value="-0.2238 -0.1824 -0.0838" />
+  <xacro:property name="chassis_sway_fwd" value="0.3776 0 -0.0838" />
+  <xacro:property name="chassis_sway_aft" value="-0.3744 0 -0.0838" />
+  <xacro:property name="chassis_heave_port_fwd" value="0.2824 0.1824 -0.0033" />
+  <xacro:property name="chassis_heave_stbd_fwd" value="0.2824 -0.1824 -0.0033" />
+  <xacro:property name="chassis_heave_port_aft" value="-0.2724 0.1824 -0.0033" />
+  <xacro:property name="chassis_heave_stbd_aft" value="-0.2724 -0.1824 -0.0033" />
+  <xacro:property name="housing_com" value="-0.0251 0.0002 -0.0224" />
+  <xacro:property name="chassis_com" value="0.0129 0 0.0561" />
+  <xacro:property name="acoustics_com" value="0.0027 0.0027 -0.0265" />
+  <xacro:property name="pneumatics_com" value="0.0141 0.0015 -0.0392" />
+  <xacro:property name="port_battery_com" value="0.0936 0.0278 -0.0003" />
+  <xacro:property name="stbd_battery_com" value="0.0962 -0.0291 -0.0003" />
+  <xacro:property name="thruster_com" value="0.0075 -0.0006 0" />
+  <xacro:property name="housing_mass" value="9.59" />
+  <xacro:property name="chassis_mass" value="2.71" />
+  <xacro:property name="acoustics_mass" value="0.97" />
+  <xacro:property name="pneumatics_mass" value="1.3503" />
+  <xacro:property name="port_battery_mass" value="1.867" />
+  <xacro:property name="stbd_battery_mass" value="1.867" />
+  <xacro:property name="thruster_mass" value="0.35" />
+  <xacro:property name="housing_inertia"><inertia ixx="0.1027" ixy="0.0000" ixz="0.0000" iyy="0.4425" iyz="0.0000" izz="0.4273" /></xacro:property>
+  <xacro:property name="chassis_inertia"><inertia ixx="0.216" ixy="0.0000" ixz="0.0000" iyy="0.1953" iyz="0.0000" izz="0.0952" /></xacro:property>
+  <xacro:property name="acoustics_inertia"><inertia ixx="0.0019" ixy="0.0000" ixz="0.0000" iyy="0.0019" iyz="0.0000" izz="0.003" /></xacro:property>
+  <xacro:property name="pneumatics_inertia"><inertia ixx="0.008" ixy="0.0000" ixz="0.0000" iyy="0.0088" iyz="0.0000" izz="0.0107" /></xacro:property>
+  <xacro:property name="port_battery_inertia"><inertia ixx="0.0034" ixy="0.0000" ixz="0.0000" iyy="0.0253" iyz="0.0000" izz="0.0262" /></xacro:property>
+  <xacro:property name="stbd_battery_inertia"><inertia ixx="0.0034" ixy="0.0000" ixz="0.0000" iyy="0.0253" iyz="0.0000" izz="0.0262" /></xacro:property>
+  <xacro:property name="thruster_inertia"><inertia ixx="0.00033" ixy="0.0000" ixz="0.0000" iyy="0.00031" iyz="0.0000" izz="0.00032" /></xacro:property>
+  <xacro:property name="housing_mesh" value="package://riptide_description/meshes/riptide_housing.stl" />
+  <xacro:property name="chassis_mesh" value="package://riptide_description/meshes/riptide_chassis.stl" />
+  <xacro:property name="acoustics_mesh" value="package://riptide_description/meshes/riptide_acoustics.stl" />
+  <xacro:property name="pneumatics_mesh" value="package://riptide_description/meshes/riptide_pneumatics.stl" />
+  <xacro:property name="port_battery_mesh" value="package://riptide_description/meshes/riptide_port_battery.stl" />
+  <xacro:property name="stbd_battery_mesh" value="package://riptide_description/meshes/riptide_stbd_battery.stl" />
+  <xacro:property name="thruster_mesh" value="package://riptide_description/meshes/blue_robotics_t200.stl" />
+</robot>

File: riptide_description/urdf/t200_thrusters.urdf.xacro (robot description, xacro)
@@ -28,5 +28,5 @@
           <mesh filename="package://riptide_description/meshes/blue_robotics_t200.stl"/>
         </geometry>
-        <material name="thruster"/>
+        <material name="housing"/>
       </visual>
       <collision>
