Commit message: Complete URDF for housings.

File: riptide_description/urdf/riptide.urdf (robot description, URDF)
Before this commit: robot riptide, 17 links, 16 joints
Links:
- removed link heave_port_aft_thruster
- removed link heave_port_fwd_thruster
- removed link heave_stbd_aft_thruster
- removed link heave_stbd_fwd_thruster
- removed link surge_port_hi_thruster
- removed link surge_port_lo_thruster
- removed link surge_stbd_hi_thruster
- removed link surge_stbd_lo_thruster
- removed link sway_aft_thruster
- removed link sway_fwd_thruster
- added link heave_port_aft_link, mass 0.35; collision mesh filename=package://riptide_description/meshes/blue_robotics_t200.stl; visual mesh filename=package://riptide_description/meshes/blue_robotics_t200.stl
- added link heave_port_fwd_link, mass 0.35; collision mesh filename=package://riptide_description/meshes/blue_robotics_t200.stl; visual mesh filename=package://riptide_description/meshes/blue_robotics_t200.stl
- added link heave_stbd_aft_link, mass 0.35; collision mesh filename=package://riptide_description/meshes/blue_robotics_t200.stl; visual mesh filename=package://riptide_description/meshes/blue_robotics_t200.stl
- added link heave_stbd_fwd_link, mass 0.35; collision mesh filename=package://riptide_description/meshes/blue_robotics_t200.stl; visual mesh filename=package://riptide_description/meshes/blue_robotics_t200.stl
- added link surge_port_hi_link, mass 0.35; collision mesh filename=package://riptide_description/meshes/blue_robotics_t200.stl; visual mesh filename=package://riptide_description/meshes/blue_robotics_t200.stl
- added link surge_port_lo_link, mass 0.35; collision mesh filename=package://riptide_description/meshes/blue_robotics_t200.stl; visual mesh filename=package://riptide_description/meshes/blue_robotics_t200.stl
- added link surge_stbd_hi_link, mass 0.35; collision mesh filename=package://riptide_description/meshes/blue_robotics_t200.stl; visual mesh filename=package://riptide_description/meshes/blue_robotics_t200.stl
- added link surge_stbd_lo_link, mass 0.35; collision mesh filename=package://riptide_description/meshes/blue_robotics_t200.stl; visual mesh filename=package://riptide_description/meshes/blue_robotics_t200.stl
- added link sway_aft_link, mass 0.35; collision mesh filename=package://riptide_description/meshes/blue_robotics_t200.stl; visual mesh filename=package://riptide_description/meshes/blue_robotics_t200.stl
- added link sway_fwd_link, mass 0.35; collision mesh filename=package://riptide_description/meshes/blue_robotics_t200.stl; visual mesh filename=package://riptide_description/meshes/blue_robotics_t200.stl
Joints:
- removed joint base_housing
- removed joint chassis_acoustics
- removed joint chassis_pneumatics
- removed joint chassis_port_battery
- removed joint chassis_stbd_battery
- removed joint heave_port_aft_thruster_joint
- removed joint heave_port_fwd_thruster_joint
- removed joint heave_stbd_aft_thruster_joint
- removed joint heave_stbd_fwd_thruster_joint
- removed joint housing_chassis
- removed joint surge_port_hi_thruster_joint
- removed joint surge_port_lo_thruster_joint
- removed joint surge_stbd_hi_thruster_joint
- removed joint surge_stbd_lo_thruster_joint
- removed joint sway_aft_thruster_joint
- removed joint sway_fwd_thruster_joint
- added joint base_housing_joint: type fixed, parent base_link, child housing_link, origin xyz=0.0737 0.0005 0.0621 rpy=0 0 0
- added joint chassis_acoustics_joint: type fixed, parent chassis_link, child acoustics_link, origin xyz=0.1699 0 -0.0584 rpy=0 0 0
- added joint chassis_pneumatics_joint: type fixed, parent chassis_link, child pneumatics_link, origin xyz=-0.1172 0 -0.0584 rpy=0 0 0
- added joint chassis_port_battery_joint: type fixed, parent chassis_link, child port_battery_link, origin xyz=-0.1781 0.1302 -0.014 rpy=0 0 0
- added joint chassis_stbd_battery_joint: type fixed, parent chassis_link, child stbd_battery_link, origin xyz=-0.1781 -0.1302 -0.014 rpy=0 0 0
- added joint heave_port_aft_joint: type fixed, parent chassis_link, child heave_port_aft_link, origin xyz=-0.2724 0.1824 -0.0033 rpy=0 0 3.14159266
- added joint heave_port_fwd_joint: type fixed, parent chassis_link, child heave_port_fwd_link, origin xyz=0.2824 0.1824 -0.0033 rpy=0 0 3.14159266
- added joint heave_stbd_aft_joint: type fixed, parent chassis_link, child heave_stbd_aft_link, origin xyz=-0.2724 -0.1824 -0.0033 rpy=0 0 0
- added joint heave_stbd_fwd_joint: type fixed, parent chassis_link, child heave_stbd_fwd_link, origin xyz=0.2824 -0.1824 -0.0033 rpy=0 0 0
- added joint housing_chassis_joint: type fixed, parent housing_link, child chassis_link, origin xyz=-0.0556 0 -0.0749 rpy=0 0 0
- added joint surge_port_hi_joint: type fixed, parent chassis_link, child surge_port_hi_link, origin xyz=-0.2238 0.1824 0.1384 rpy=0 -1.57079633 3.14159266
- added joint surge_port_lo_joint: type fixed, parent chassis_link, child surge_port_lo_link, origin xyz=-0.2238 0.1824 -0.0838 rpy=0 -1.57079633 3.14159266
- added joint surge_stbd_hi_joint: type fixed, parent chassis_link, child surge_stbd_hi_link, origin xyz=-0.2238 -0.1824 0.1384 rpy=0 1.57079633 0
- added joint surge_stbd_lo_joint: type fixed, parent chassis_link, child surge_stbd_lo_link, origin xyz=-0.2238 -0.1824 -0.0838 rpy=0 1.57079633 0
- added joint sway_aft_joint: type fixed, parent chassis_link, child sway_aft_link, origin xyz=-0.3744 0 -0.0838 rpy=0 -1.57079633 -1.57079633
- added joint sway_fwd_joint: type fixed, parent chassis_link, child sway_fwd_link, origin xyz=0.3776 0 -0.0838 rpy=0 1.57079633 1.57079633

File: riptide_description/urdf/riptide.urdf.xacro (robot description, xacro)
@@ -7,16 +7,25 @@
 <!--                                  -->
 <robot name="riptide" xmlns:xacro="http://ros.org/wiki/xacro">
+  <xacro:property name="M_PI" value="3.14159266"/>
   <xacro:include filename="riptide_dimensions.urdf.xacro" />
   <xacro:include filename="riptide_links.urdf.xacro" />
   <xacro:include filename="riptide_joints.urdf.xacro" />
-  <xacro:include filename="t200_thruster.urdf.xacro" />
+  <material name="housing">
+    <color rgba="0.36 0.24 0.24 1.0"/>
+  </material>
   <material name="chassis">
-    <color rgba="0 0 0 1.0"/>
+    <color rgba="0.06 0.06 0.06 1.0"/>
   </material>
-  <material name="housing">
-    <color rgba="0.2 0.2 0.2 1.0"/>
+  <material name="acoustics">
+    <color rgba="0.12 0.12 0.12 1.0"/>
+  </material>
+  <material name="pneumatics">
+    <color rgba="0.12 0.12 0.12 1.0"/>
+  </material>
+  <material name="battery">
+    <color rgba="0.12 0.12 0.12 1.0"/>
   </material>
   <material name="thruster">
-    <color rgba="0.365 0 0 1.0"/>
+    <color rgba="0.36 0.36 0.36 1.0"/>
   </material>
 </robot>

File: riptide_description/urdf/riptide_dimensions.urdf.xacro (robot description, xacro)
@@ -1,5 +1,4 @@
 <?xml version="1.0"?>
 <robot xmlns:xacro="http://ros.org/wiki/xacro">
-  <xacro:property name="M_PI" value="3.14159266"/>
   <xacro:property name="housing_camera_port" value="0.2744 0.04 -0.0004" />
   <xacro:property name="housing_camera_stbd" value="0.2744 -0.04 -0.0004" />
@@ -15,5 +14,5 @@
   <xacro:property name="chassis_stbd_battery" value="-0.1781 -0.1302 -0.014" />
   <xacro:property name="chassis_surge_port_hi" value="-0.2238 0.1824 0.1384" />
-  <xacro:property name="chassis_surge_port_lo" value="-0.2238 -0.1824 0.1384" />
+  <xacro:property name="chassis_surge_stbd_hi" value="-0.2238 -0.1824 0.1384" />
   <xacro:property name="chassis_surge_port_lo" value="-0.2238 0.1824 -0.0838" />
   <xacro:property name="chassis_surge_stbd_lo" value="-0.2238 -0.1824 -0.0838" />
@@ -52,3 +51,13 @@
   <xacro:property name="stbd_battery_mesh" value="package://riptide_description/meshes/riptide_stbd_battery.stl" />
   <xacro:property name="thruster_mesh" value="package://riptide_description/meshes/blue_robotics_t200.stl" />
+  <xacro:property name="align_surge_port_hi" value="0 ${-M_PI/2} ${M_PI}" />
+  <xacro:property name="align_surge_stbd_hi" value="0 ${M_PI/2} 0" />
+  <xacro:property name="align_surge_port_lo" value="0 ${-M_PI/2} ${M_PI}" />
+  <xacro:property name="align_surge_stbd_lo" value="0 ${M_PI/2} 0" />
+  <xacro:property name="align_sway_fwd" value="0 ${M_PI/2} ${M_PI/2}" />
+  <xacro:property name="align_sway_aft" value="0 ${-M_PI/2} ${-M_PI/2}" />
+  <xacro:property name="align_heave_port_fwd" value="0 0 ${M_PI}" />
+  <xacro:property name="align_heave_stbd_fwd" value="0 0 0" />
+  <xacro:property name="align_heave_port_aft" value="0 0 ${M_PI}" />
+  <xacro:property name="align_heave_stbd_aft" value="0 0 0" />
 </robot>

File: riptide_description/urdf/riptide_joints.urdf.xacro (robot description, xacro)
@@ -1,33 +1,56 @@
 <?xml version="1.0"?>
 <robot xmlns:xacro="http://ros.org/wiki/xacro">
-  <joint name="base_housing" type="fixed">
+  <!--                -->
+  <!-- Housing Joints -->
+  <!--                -->
+  <joint name="base_housing_joint" type="fixed">
     <origin xyz="${base_housing}" rpy="0 0 0"/>
     <parent link="base_link"/>
     <child link="housing_link"/>
   </joint>
-  <joint name="housing_chassis" type="fixed">
+  <joint name="housing_chassis_joint" type="fixed">
     <origin xyz="${housing_chassis}" rpy="0 0 0"/>
     <parent link="housing_link"/>
     <child link="chassis_link"/>
   </joint>
-  <joint name="chassis_acoustics" type="fixed">
+  <joint name="chassis_acoustics_joint" type="fixed">
     <origin xyz="${chassis_acoustics}" rpy="0 0 0"/>
     <parent link="chassis_link"/>
     <child link="acoustics_link"/>
   </joint>
-  <joint name="chassis_pneumatics" type="fixed">
+  <joint name="chassis_pneumatics_joint" type="fixed">
     <origin xyz="${chassis_pneumatics}" rpy="0 0 0"/>
     <parent link="chassis_link"/>
     <child link="pneumatics_link"/>
   </joint>
-  <joint name="chassis_port_battery" type="fixed">
+  <joint name="chassis_port_battery_joint" type="fixed">
     <origin xyz="${chassis_port_battery}" rpy="0 0 0"/>
     <parent link="chassis_link"/>
     <child link="port_battery_link"/>
   </joint>
-  <joint name="chassis_stbd_battery" type="fixed">
+  <joint name="chassis_stbd_battery_joint" type="fixed">
     <origin xyz="${chassis_stbd_battery}" rpy="0 0 0"/>
     <parent link="chassis_link"/>
     <child link="stbd_battery_link"/>
   </joint>
+  <!--                 -->
+  <!-- Thruster Joints -->
+  <!--                 -->
+  <xacro:macro name="thruster_joint" params="name p o">
+    <joint name="${name}_joint" type="fixed">
+      <origin xyz="${p}" rpy="${o}"/>
+      <parent link="chassis_link"/>
+      <child link="${name}_link"/>
+    </joint>
+  </xacro:macro>
+  <xacro:thruster_joint name="surge_port_hi" p="${chassis_surge_port_hi}" o="${align_surge_port_hi}"/>
+  <xacro:thruster_joint name="surge_stbd_hi" p="${chassis_surge_stbd_hi}" o="${align_surge_stbd_hi}"/>
+  <xacro:thruster_joint name="surge_port_lo" p="${chassis_surge_port_lo}" o="${align_surge_port_lo}"/>
+  <xacro:thruster_joint name="surge_stbd_lo" p="${chassis_surge_stbd_lo}" o="${align_surge_stbd_lo}"/>
+  <xacro:thruster_joint name="sway_fwd" p="${chassis_sway_fwd}" o="${align_sway_fwd}"/>
+  <xacro:thruster_joint name="sway_aft" p="${chassis_sway_aft}" o="${align_sway_aft}"/>
+  <xacro:thruster_joint name="heave_port_fwd" p="${chassis_heave_port_fwd}" o="${align_heave_port_fwd}"/>
+  <xacro:thruster_joint name="heave_stbd_fwd" p="${chassis_heave_stbd_fwd}" o="${align_heave_stbd_fwd}"/>
+  <xacro:thruster_joint name="heave_port_aft" p="${chassis_heave_port_aft}" o="${align_heave_port_aft}"/>
+  <xacro:thruster_joint name="heave_stbd_aft" p="${chassis_heave_stbd_aft}" o="${align_heave_stbd_aft}"/>
 </robot>

File: riptide_description/urdf/riptide_links.urdf.xacro (robot description, xacro)
@@ -1,4 +1,7 @@
 <?xml version="1.0"?>
 <robot xmlns:xacro="http://ros.org/wiki/xacro">
+  <!--               -->
+  <!-- Housing Links -->
+  <!--               -->
   <link name="base_link">
   </link>
@@ -49,5 +52,5 @@
         <mesh filename="${acoustics_mesh}" />
       </geometry>
-      <material name="housing" />
+      <material name="acoustics" />
     </visual>
     <collision>
@@ -67,5 +70,5 @@
         <mesh filename="${pneumatics_mesh}" />
       </geometry>
-      <material name="housing" />
+      <material name="pneumatics" />
     </visual>
     <collision>
@@ -85,5 +88,5 @@
         <mesh filename="${port_battery_mesh}" />
       </geometry>
-      <material name="housing" />
+      <material name="battery" />
     </visual>
     <collision>
@@ -103,5 +106,5 @@
         <mesh filename="${stbd_battery_mesh}" />
       </geometry>
-        <material name="housing"/>
+        <material name="battery"/>
     </visual>
     <collision>
@@ -111,3 +114,36 @@
     </collision>
   </link>
+  <!--                -->
+  <!-- Thruster Links -->
+  <!--                -->
+  <xacro:macro name="thruster_link" params="name">
+    <link name="${name}_link">
+      <inertial>
+        <origin xyz="${thruster_com}" rpy="0 0 0" />
+        <mass value="${thruster_mass}" />
+        <xacro:insert_block name="thruster_inertia" />
+      </inertial>
+      <visual>
+        <geometry>
+          <mesh filename="${thruster_mesh}" />
+        </geometry>
+          <material name="thruster"/>
+      </visual>
+      <collision>
+        <geometry>
+          <mesh filename="${thruster_mesh}" />
+        </geometry>
+      </collision>
+    </link>
+  </xacro:macro>
+  <xacro:thruster_link name="surge_port_hi" />
+  <xacro:thruster_link name="surge_stbd_hi" />
+  <xacro:thruster_link name="surge_port_lo" />
+  <xacro:thruster_link name="surge_stbd_lo" />
+  <xacro:thruster_link name="sway_fwd" />
+  <xacro:thruster_link name="sway_aft" />
+  <xacro:thruster_link name="heave_port_fwd" />
+  <xacro:thruster_link name="heave_stbd_fwd" />
+  <xacro:thruster_link name="heave_port_aft" />
+  <xacro:thruster_link name="heave_stbd_aft" />
 </robot>
