Commit message: Update housing properties and mesh names.

File: riptide_description/urdf/riptide.urdf (robot description, URDF)
Before this commit: robot riptide, 17 links, 16 joints
Links:
- link acoustics_link: geometry collision mesh filename=package://riptide_description/meshes/acoustics.stl; visual mesh filename=package://riptide_description/meshes/acoustics.stl
- link chassis_link: geometry collision mesh filename=package://riptide_description/meshes/chassis.stl; visual mesh filename=package://riptide_description/meshes/chassis.stl
- link heave_port_aft_link: geometry collision mesh filename=package://riptide_description/meshes/thruster.stl; visual mesh filename=package://riptide_description/meshes/thruster.stl
- link heave_port_fwd_link: geometry collision mesh filename=package://riptide_description/meshes/thruster.stl; visual mesh filename=package://riptide_description/meshes/thruster.stl
- link heave_stbd_aft_link: geometry collision mesh filename=package://riptide_description/meshes/thruster.stl; visual mesh filename=package://riptide_description/meshes/thruster.stl
- link heave_stbd_fwd_link: geometry collision mesh filename=package://riptide_description/meshes/thruster.stl; visual mesh filename=package://riptide_description/meshes/thruster.stl
- link housing_link: mass 9.59 -> 13.87; geometry collision mesh filename=package://riptide_description/meshes/housing.stl; visual mesh filename=package://riptide_description/meshes/housing.stl
- link pneumatics_link: geometry collision mesh filename=package://riptide_description/meshes/pneumatics.stl; visual mesh filename=package://riptide_description/meshes/pneumatics.stl
- link port_battery_link: geometry collision mesh filename=package://riptide_description/meshes/port_battery.stl; visual mesh filename=package://riptide_description/meshes/port_battery.stl
- link stbd_battery_link: geometry collision mesh filename=package://riptide_description/meshes/stbd_battery.stl; visual mesh filename=package://riptide_description/meshes/stbd_battery.stl
- link surge_port_hi_link: geometry collision mesh filename=package://riptide_description/meshes/thruster.stl; visual mesh filename=package://riptide_description/meshes/thruster.stl
- link surge_port_lo_link: geometry collision mesh filename=package://riptide_description/meshes/thruster.stl; visual mesh filename=package://riptide_description/meshes/thruster.stl
- link surge_stbd_hi_link: geometry collision mesh filename=package://riptide_description/meshes/thruster.stl; visual mesh filename=package://riptide_description/meshes/thruster.stl
- link surge_stbd_lo_link: geometry collision mesh filename=package://riptide_description/meshes/thruster.stl; visual mesh filename=package://riptide_description/meshes/thruster.stl
- link sway_aft_link: geometry collision mesh filename=package://riptide_description/meshes/thruster.stl; visual mesh filename=package://riptide_description/meshes/thruster.stl
- link sway_fwd_link: geometry collision mesh filename=package://riptide_description/meshes/thruster.stl; visual mesh filename=package://riptide_description/meshes/thruster.stl
Joints:
- joint chassis_acoustics_joint: origin xyz=0.1699 0 -0.0584 rpy=0 0 0 -> xyz=-0.1699 0.0000 0.0584 rpy=0 0 0
- joint chassis_pneumatics_joint: origin xyz=-0.1172 0 -0.0584 rpy=0 0 0 -> xyz=0.1172 0.0000 0.0584 rpy=0 0 0
- joint chassis_port_battery_joint: origin xyz=-0.1781 0.1302 -0.014 rpy=0 0 0 -> xyz=0.1781 -0.1302 0.0140 rpy=0 0 0
- joint chassis_stbd_battery_joint: origin xyz=-0.1781 -0.1302 -0.014 rpy=0 0 0 -> xyz=0.1781 0.1302 0.0140 rpy=0 0 0
- joint housing_chassis_joint: origin xyz=-0.0556 0 -0.0749 rpy=0 0 0 -> xyz=-0.0556 0.0000 -0.0749 rpy=0 0 0
- joint sway_aft_joint: origin xyz=-0.3744 0 -0.0838 rpy=0 -1.57079633 -1.57079633 -> xyz=-0.3744 0.0000 -0.0838 rpy=0 -1.57079633 -1.57079633
- joint sway_fwd_joint: origin xyz=0.3776 0 -0.0838 rpy=0 1.57079633 1.57079633 -> xyz=0.3776 0.0000 -0.0838 rpy=0 1.57079633 1.57079633

File: riptide_description/urdf/riptide_dimensions.urdf.xacro (robot description, xacro)
@@ -1,54 +1,54 @@
 <?xml version="1.0"?>
 <robot xmlns:xacro="http://ros.org/wiki/xacro">
-  <xacro:property name="housing_camera_port" value="0.2744 0.04 -0.0004" />
-  <xacro:property name="housing_camera_stbd" value="0.2744 -0.04 -0.0004" />
-  <xacro:property name="housing_camera_down" value="0.236 0 -0.062" />
-  <xacro:property name="housing_depth_sensor" value="0 0 0.1049" />
+  <xacro:property name="housing_camera_port" value="0.2744 0.0400 -0.0004" />
+  <xacro:property name="housing_camera_stbd" value="0.2744 -0.0400 -0.0004" />
+  <xacro:property name="housing_camera_down" value="0.2360 0.0000 -0.0620" />
+  <xacro:property name="housing_depth_sensor" value="0.0000 0.0000 0.1049" />
   <xacro:property name="housing_imu_one" value="0.1322 -0.0056 0.0268" />
   <xacro:property name="housing_imu_two" value="-0.1469 0.0004 -0.0405" />
   <xacro:property name="base_housing" value="0.0737 0.0005 0.0621" />
-  <xacro:property name="housing_chassis" value="-0.0556 0 -0.0749" />
-  <xacro:property name="chassis_acoustics" value="0.1699 0 -0.0584" />
-  <xacro:property name="chassis_pneumatics" value="-0.1172 0 -0.0584" />
-  <xacro:property name="chassis_port_battery" value="-0.1781 0.1302 -0.014" />
-  <xacro:property name="chassis_stbd_battery" value="-0.1781 -0.1302 -0.014" />
+  <xacro:property name="housing_chassis" value="-0.0556 0.0000 -0.0749" />
+  <xacro:property name="chassis_acoustics" value="0.1699 0.0000 -0.0584" />
+  <xacro:property name="chassis_pneumatics" value="-0.1172 0.0000 -0.0584" />
+  <xacro:property name="chassis_port_battery" value="-0.1781 0.1302 -0.0140" />
+  <xacro:property name="chassis_stbd_battery" value="-0.1781 -0.1302 -0.0140" />
   <xacro:property name="chassis_surge_port_hi" value="-0.2238 0.1824 0.1384" />
   <xacro:property name="chassis_surge_stbd_hi" value="-0.2238 -0.1824 0.1384" />
   <xacro:property name="chassis_surge_port_lo" value="-0.2238 0.1824 -0.0838" />
   <xacro:property name="chassis_surge_stbd_lo" value="-0.2238 -0.1824 -0.0838" />
-  <xacro:property name="chassis_sway_fwd" value="0.3776 0 -0.0838" />
-  <xacro:property name="chassis_sway_aft" value="-0.3744 0 -0.0838" />
+  <xacro:property name="chassis_sway_fwd" value="0.3776 0.0000 -0.0838" />
+  <xacro:property name="chassis_sway_aft" value="-0.3744 0.0000 -0.0838" />
   <xacro:property name="chassis_heave_port_fwd" value="0.2824 0.1824 -0.0033" />
   <xacro:property name="chassis_heave_stbd_fwd" value="0.2824 -0.1824 -0.0033" />
   <xacro:property name="chassis_heave_port_aft" value="-0.2724 0.1824 -0.0033" />
   <xacro:property name="chassis_heave_stbd_aft" value="-0.2724 -0.1824 -0.0033" />
-  <xacro:property name="housing_com" value="-0.0251 0.0002 -0.0224" />
-  <xacro:property name="chassis_com" value="0.0129 0 0.0561" />
+  <xacro:property name="housing_com" value="-0.0434 0.0009 -0.0158" />
+  <xacro:property name="chassis_com" value="0.0129 0.0000 0.0561" />
   <xacro:property name="acoustics_com" value="0.0027 0.0027 -0.0265" />
   <xacro:property name="pneumatics_com" value="0.0141 0.0015 -0.0392" />
   <xacro:property name="port_battery_com" value="0.0936 0.0278 -0.0003" />
   <xacro:property name="stbd_battery_com" value="0.0962 -0.0291 -0.0003" />
-  <xacro:property name="thruster_com" value="0.0075 -0.0006 0" />
-  <xacro:property name="housing_mass" value="9.59" />
-  <xacro:property name="chassis_mass" value="2.71" />
-  <xacro:property name="acoustics_mass" value="0.97" />
+  <xacro:property name="thruster_com" value="0.0075 -0.0006 0.0000" />
+  <xacro:property name="housing_mass" value="13.8700" />
+  <xacro:property name="chassis_mass" value="2.7100" />
+  <xacro:property name="acoustics_mass" value="0.9700" />
   <xacro:property name="pneumatics_mass" value="1.3503" />
-  <xacro:property name="port_battery_mass" value="1.867" />
-  <xacro:property name="stbd_battery_mass" value="1.867" />
-  <xacro:property name="thruster_mass" value="0.35" />
-  <xacro:property name="housing_inertia"><inertia ixx="0.1027" ixy="0.0000" ixz="0.0000" iyy="0.4425" iyz="0.0000" izz="0.4273" /></xacro:property>
-  <xacro:property name="chassis_inertia"><inertia ixx="0.216" ixy="0.0000" ixz="0.0000" iyy="0.1953" iyz="0.0000" izz="0.0952" /></xacro:property>
-  <xacro:property name="acoustics_inertia"><inertia ixx="0.0019" ixy="0.0000" ixz="0.0000" iyy="0.0019" iyz="0.0000" izz="0.003" /></xacro:property>
-  <xacro:property name="pneumatics_inertia"><inertia ixx="0.008" ixy="0.0000" ixz="0.0000" iyy="0.0088" iyz="0.0000" izz="0.0107" /></xacro:property>
+  <xacro:property name="port_battery_mass" value="1.8670" />
+  <xacro:property name="stbd_battery_mass" value="1.8670" />
+  <xacro:property name="thruster_mass" value="0.3500" />
+  <xacro:property name="housing_inertia"><inertia ixx="0.1187" ixy="0.0000" ixz="0.0000" iyy="0.6524" iyz="0.0000" izz="0.6379" /></xacro:property>
+  <xacro:property name="chassis_inertia"><inertia ixx="0.2160" ixy="0.0000" ixz="0.0000" iyy="0.1953" iyz="0.0000" izz="0.0952" /></xacro:property>
+  <xacro:property name="acoustics_inertia"><inertia ixx="0.0019" ixy="0.0000" ixz="0.0000" iyy="0.0019" iyz="0.0000" izz="0.0030" /></xacro:property>
+  <xacro:property name="pneumatics_inertia"><inertia ixx="0.0080" ixy="0.0000" ixz="0.0000" iyy="0.0088" iyz="0.0000" izz="0.0107" /></xacro:property>
   <xacro:property name="port_battery_inertia"><inertia ixx="0.0034" ixy="0.0000" ixz="0.0000" iyy="0.0253" iyz="0.0000" izz="0.0262" /></xacro:property>
   <xacro:property name="stbd_battery_inertia"><inertia ixx="0.0034" ixy="0.0000" ixz="0.0000" iyy="0.0253" iyz="0.0000" izz="0.0262" /></xacro:property>
-  <xacro:property name="thruster_inertia"><inertia ixx="0.00033" ixy="0.0000" ixz="0.0000" iyy="0.00031" iyz="0.0000" izz="0.00032" /></xacro:property>
-  <xacro:property name="housing_mesh" value="package://riptide_description/meshes/riptide_housing.stl" />
-  <xacro:property name="chassis_mesh" value="package://riptide_description/meshes/riptide_chassis.stl" />
-  <xacro:property name="acoustics_mesh" value="package://riptide_description/meshes/riptide_acoustics.stl" />
-  <xacro:property name="pneumatics_mesh" value="package://riptide_description/meshes/riptide_pneumatics.stl" />
-  <xacro:property name="port_battery_mesh" value="package://riptide_description/meshes/riptide_port_battery.stl" />
-  <xacro:property name="stbd_battery_mesh" value="package://riptide_description/meshes/riptide_stbd_battery.stl" />
-  <xacro:property name="thruster_mesh" value="package://riptide_description/meshes/blue_robotics_t200.stl" />
+  <xacro:property name="thruster_inertia"><inertia ixx="0.0003" ixy="0.0000" ixz="0.0000" iyy="0.0003" iyz="0.0000" izz="0.0003" /></xacro:property>
+  <xacro:property name="housing_mesh" value="package://riptide_description/meshes/housing.stl" />
+  <xacro:property name="chassis_mesh" value="package://riptide_description/meshes/chassis.stl" />
+  <xacro:property name="acoustics_mesh" value="package://riptide_description/meshes/acoustics.stl" />
+  <xacro:property name="pneumatics_mesh" value="package://riptide_description/meshes/pneumatics.stl" />
+  <xacro:property name="port_battery_mesh" value="package://riptide_description/meshes/port_battery.stl" />
+  <xacro:property name="stbd_battery_mesh" value="package://riptide_description/meshes/stbd_battery.stl" />
+  <xacro:property name="thruster_mesh" value="package://riptide_description/meshes/thruster.stl" />
   <xacro:property name="align_surge_port_hi" value="0 ${-M_PI/2} ${M_PI}" />
   <xacro:property name="align_surge_stbd_hi" value="0 ${M_PI/2} 0" />

Commit message: Riptide is no longer entering orbit.

File: riptide_description/urdf/riptide.urdf (robot description, URDF)
Before this commit: robot riptide, 17 links, 16 joints
Joints:
- joint chassis_acoustics_joint: origin xyz=-0.1699 0.0000 0.0584 rpy=0 0 0 -> xyz=0.1699 0.0000 -0.0584 rpy=0 0 0
- joint chassis_pneumatics_joint: origin xyz=0.1172 0.0000 0.0584 rpy=0 0 0 -> xyz=-0.1172 0.0000 -0.0584 rpy=0 0 0
- joint chassis_port_battery_joint: origin xyz=0.1781 -0.1302 0.0140 rpy=0 0 0 -> xyz=-0.1781 0.1302 -0.0140 rpy=0 0 0
- joint chassis_stbd_battery_joint: origin xyz=0.1781 0.1302 0.0140 rpy=0 0 0 -> xyz=-0.1781 -0.1302 -0.0140 rpy=0 0 0

File: riptide_description/urdf/riptide_links.urdf.xacro (robot description, xacro)
@@ -117,6 +117,6 @@
   <!-- Thruster Links -->
   <!--                -->
-  <xacro:macro name="thruster_link" params="name">
-    <link name="${name}_link">
+  <xacro:macro name="thruster_link" params="thruster">
+    <link name="${thruster}_link">
       <inertial>
         <origin xyz="${thruster_com}" rpy="0 0 0" />
@@ -137,13 +137,13 @@
     </link>
   </xacro:macro>
-  <xacro:thruster_link name="surge_port_hi" />
-  <xacro:thruster_link name="surge_stbd_hi" />
-  <xacro:thruster_link name="surge_port_lo" />
-  <xacro:thruster_link name="surge_stbd_lo" />
-  <xacro:thruster_link name="sway_fwd" />
-  <xacro:thruster_link name="sway_aft" />
-  <xacro:thruster_link name="heave_port_fwd" />
-  <xacro:thruster_link name="heave_stbd_fwd" />
-  <xacro:thruster_link name="heave_port_aft" />
-  <xacro:thruster_link name="heave_stbd_aft" />
+  <xacro:thruster_link thruster="surge_port_hi" />
+  <xacro:thruster_link thruster="surge_stbd_hi" />
+  <xacro:thruster_link thruster="surge_port_lo" />
+  <xacro:thruster_link thruster="surge_stbd_lo" />
+  <xacro:thruster_link thruster="sway_fwd" />
+  <xacro:thruster_link thruster="sway_aft" />
+  <xacro:thruster_link thruster="heave_port_fwd" />
+  <xacro:thruster_link thruster="heave_stbd_fwd" />
+  <xacro:thruster_link thruster="heave_port_aft" />
+  <xacro:thruster_link thruster="heave_stbd_aft" />
 </robot>

File: riptide_description/urdf/riptide_sim.gazebo.xacro (robot description, xacro)
@@ -6,5 +6,50 @@
   <gazebo>
     <!--  Buoyancy  -->
-    <plugin name="BuoyancyPlugin" filename="libBuoyancyPlugin.so"/>
+    <plugin name="BuoyancyPlugin" filename="libBuoyancyPlugin.so">
+      <link name="base_link">
+        <center_of_volume>0 0 0</center_of_volume>
+        <volume>0.0253</volume>
+      </link>
+      <!-- <link name="housing_link">
+        <center_of_volume>0 0 0</center_of_volume>
+        <volume>0.0223</volume>
+      </link>
+      <link name="chassis_link">
+        <center_of_volume>0 0 0</center_of_volume>
+        <volume>0.0001</volume>
+      </link>
+      <link name="acoustics_link">
+        <center_of_volume>0 0 0</center_of_volume>
+        <volume>0.0004</volume>
+      </link>
+      <link name="pneumatics_link">
+        <center_of_volume>0 0 0</center_of_volume>
+        <volume>0.0005</volume>
+      </link>
+      <link name="port_battery_link">
+        <center_of_volume>0 0 0</center_of_volume>
+        <volume>0.0009</volume>
+      </link>
+      <link name="stbd_battery_link">
+        <center_of_volume>0 0 0</center_of_volume>
+        <volume>0.0009</volume>
+      </link>
+      <xacro:macro name="thruster_volume" params="thruster">
+        <link name="${thruster}_link">
+          <center_of_volume>0 0 0</center_of_volume>
+          <volume>0.0002</volume>
+        </link>
+      </xacro:macro>
+      <xacro:thruster_volume thruster="surge_port_hi" />
+      <xacro:thruster_volume thruster="surge_stbd_hi" />
+      <xacro:thruster_volume thruster="surge_port_lo" />
+      <xacro:thruster_volume thruster="surge_stbd_lo" />
+      <xacro:thruster_volume thruster="sway_fwd" />
+      <xacro:thruster_volume thruster="sway_aft" />
+      <xacro:thruster_volume thruster="heave_port_fwd" />
+      <xacro:thruster_volume thruster="heave_stbd_fwd" />
+      <xacro:thruster_volume thruster="heave_port_aft" />
+      <xacro:thruster_volume thruster="heave_stbd_aft" /> -->
+    </plugin>
   </gazebo>
     <!--             -->
