Commit message: Updated the dimensions, yay...

File: riptide_description/urdf/riptide.urdf (robot description, URDF)
Before this commit: robot riptide, 17 links, 16 joints
Links:
- link acoustics_link: mass 0.97 -> 0.9657
- link chassis_link: mass 2.71 -> 2.7134
- link heave_port_aft_link: mass 0.35 -> 0.3518
- link heave_port_fwd_link: mass 0.35 -> 0.3518
- link heave_stbd_aft_link: mass 0.35 -> 0.3518
- link heave_stbd_fwd_link: mass 0.35 -> 0.3518
- link housing_link: mass 13.87 -> 14.3153
- link port_battery_link: mass 1.867 -> 1.8671
- link stbd_battery_link: mass 1.867 -> 1.8671
- link surge_port_hi_link: mass 0.35 -> 0.3518
- link surge_port_lo_link: mass 0.35 -> 0.3518
- link surge_stbd_hi_link: mass 0.35 -> 0.3518
- link surge_stbd_lo_link: mass 0.35 -> 0.3518
- link sway_aft_link: mass 0.35 -> 0.3518
- link sway_fwd_link: mass 0.35 -> 0.3518

File: riptide_description/urdf/riptide_dimensions.urdf.xacro (robot description, xacro)
@@ -23,25 +23,39 @@
   <xacro:property name="chassis_heave_port_aft" value="-0.2724 0.1824 -0.0033" />
   <xacro:property name="chassis_heave_stbd_aft" value="-0.2724 -0.1824 -0.0033" />
-  <xacro:property name="housing_com" value="-0.0434 0.0009 -0.0158" />
-  <xacro:property name="chassis_com" value="0.0129 0.0000 0.0561" />
+  <xacro:property name="housing_com" value="-0.0434 0.0009 -0.0155" />
+  <xacro:property name="chassis_com" value="-0.0129 0.0000 -0.0561" />
   <xacro:property name="acoustics_com" value="0.0027 0.0027 -0.0265" />
   <xacro:property name="pneumatics_com" value="0.0141 0.0015 -0.0392" />
   <xacro:property name="port_battery_com" value="0.0936 0.0278 -0.0003" />
-  <xacro:property name="stbd_battery_com" value="0.0962 -0.0291 -0.0003" />
-  <xacro:property name="thruster_com" value="0.0075 -0.0006 0.0000" />
-  <xacro:property name="housing_mass" value="13.8700" />
-  <xacro:property name="chassis_mass" value="2.7100" />
-  <xacro:property name="acoustics_mass" value="0.9700" />
+  <xacro:property name="stbd_battery_com" value="0.0936 -0.0278 -0.0003" />
+  <xacro:property name="thruster_com" value="0.0000 0.0006 0.0075" />
+  <xacro:property name="housing_mass" value="14.3153" />
+  <xacro:property name="chassis_mass" value="2.7134" />
+  <xacro:property name="acoustics_mass" value="0.9657" />
   <xacro:property name="pneumatics_mass" value="1.3503" />
-  <xacro:property name="port_battery_mass" value="1.8670" />
-  <xacro:property name="stbd_battery_mass" value="1.8670" />
-  <xacro:property name="thruster_mass" value="0.3500" />
-  <xacro:property name="housing_inertia"><inertia ixx="0.1187" ixy="0.0000" ixz="0.0000" iyy="0.6524" iyz="0.0000" izz="0.6379" /></xacro:property>
-  <xacro:property name="chassis_inertia"><inertia ixx="0.2160" ixy="0.0000" ixz="0.0000" iyy="0.1953" iyz="0.0000" izz="0.0952" /></xacro:property>
-  <xacro:property name="acoustics_inertia"><inertia ixx="0.0019" ixy="0.0000" ixz="0.0000" iyy="0.0019" iyz="0.0000" izz="0.0030" /></xacro:property>
+  <xacro:property name="port_battery_mass" value="1.8671" />
+  <xacro:property name="stbd_battery_mass" value="1.8671" />
+  <xacro:property name="thruster_mass" value="0.3518" />
+  <xacro:property name="housing_inertia"><inertia ixx="0.1230" ixy="0.0000" ixz="0.0000" iyy="0.6568" iyz="0.0000" izz="0.6422" /></xacro:property>
+  <xacro:property name="chassis_inertia"><inertia ixx="0.0572" ixy="0.0000" ixz="0.0000" iyy="0.1657" iyz="0.0000" izz="0.1830" /></xacro:property>
+  <xacro:property name="acoustics_inertia"><inertia ixx="0.0026" ixy="0.0000" ixz="0.0000" iyy="0.0026" iyz="0.0000" izz="0.0030" /></xacro:property>
   <xacro:property name="pneumatics_inertia"><inertia ixx="0.0080" ixy="0.0000" ixz="0.0000" iyy="0.0088" iyz="0.0000" izz="0.0107" /></xacro:property>
   <xacro:property name="port_battery_inertia"><inertia ixx="0.0034" ixy="0.0000" ixz="0.0000" iyy="0.0253" iyz="0.0000" izz="0.0262" /></xacro:property>
   <xacro:property name="stbd_battery_inertia"><inertia ixx="0.0034" ixy="0.0000" ixz="0.0000" iyy="0.0253" iyz="0.0000" izz="0.0262" /></xacro:property>
   <xacro:property name="thruster_inertia"><inertia ixx="0.0003" ixy="0.0000" ixz="0.0000" iyy="0.0003" iyz="0.0000" izz="0.0003" /></xacro:property>
+  <xacro:property name="housing_cov" value="-0.0480 0.0000 -0.0037" />
+  <xacro:property name="chassis_cov" value="-0.0120 0.0000 -0.0566" />
+  <xacro:property name="acoustics_cov" value="0.0014 0.0014 -0.0277" />
+  <xacro:property name="pneumatics_cov" value="0.0025 0.0002 -0.0369" />
+  <xacro:property name="port_battery_cov" value="0.1257 0.0335 -0.0001" />
+  <xacro:property name="stbd_battery_cov" value="0.1257 -0.0335 -0.0001" />
+  <xacro:property name="thruster_cov" value="0.0000 0.0006 0.0075" />
+  <xacro:property name="housing_volume" value="0.0262" />
+  <xacro:property name="chassis_volume" value="0.0010" />
+  <xacro:property name="acoustics_volume" value="0.0010" />
+  <xacro:property name="pneumatics_volume" value="0.0024" />
+  <xacro:property name="port_battery_volume" value="0.0013" />
+  <xacro:property name="stbd_battery_volume" value="0.0013" />
+  <xacro:property name="thruster_volume" value="0.0002" />
   <xacro:property name="housing_mesh" value="package://riptide_description/meshes/housing.stl" />
   <xacro:property name="chassis_mesh" value="package://riptide_description/meshes/chassis.stl" />

File: riptide_description/urdf/riptide_sim.gazebo.xacro (robot description, xacro)
@@ -9,34 +9,34 @@
       <link name="base_link">
         <center_of_volume>0 0 0</center_of_volume>
-        <volume>0.0253</volume>
+        <volume>0</volume>
       </link>
-      <!-- <link name="housing_link">
-        <center_of_volume>0 0 0</center_of_volume>
-        <volume>0.0223</volume>
+      <link name="housing_link">
+        <center_of_volume>${housing_cov}</center_of_volume>
+        <volume>${housing_volume}</volume>
       </link>
       <link name="chassis_link">
-        <center_of_volume>0 0 0</center_of_volume>
-        <volume>0.0001</volume>
+        <center_of_volume>${chassis_cov}</center_of_volume>
+        <volume>${chassis_volume}</volume>
       </link>
       <link name="acoustics_link">
-        <center_of_volume>0 0 0</center_of_volume>
-        <volume>0.0004</volume>
+        <center_of_volume>${acoustics_cov}</center_of_volume>
+        <volume>${acoustics_volume}</volume>
       </link>
       <link name="pneumatics_link">
-        <center_of_volume>0 0 0</center_of_volume>
-        <volume>0.0005</volume>
+        <center_of_volume>${pneumatics_cov}</center_of_volume>
+        <volume>${pneumatics_volume}</volume>
       </link>
       <link name="port_battery_link">
-        <center_of_volume>0 0 0</center_of_volume>
-        <volume>0.0009</volume>
+        <center_of_volume>${port_battery_cov}</center_of_volume>
+        <volume>${port_battery_volume}</volume>
       </link>
       <link name="stbd_battery_link">
-        <center_of_volume>0 0 0</center_of_volume>
-        <volume>0.0009</volume>
+        <center_of_volume>${stbd_battery_cov}</center_of_volume>
+        <volume>${stbd_battery_volume}</volume>
       </link>
       <xacro:macro name="thruster_volume" params="thruster">
         <link name="${thruster}_link">
-          <center_of_volume>0 0 0</center_of_volume>
-          <volume>0.0002</volume>
+          <center_of_volume>${thruster_cov}</center_of_volume>
+          <volume>${thruster_volume}</volume>
         </link>
       </xacro:macro>
@@ -50,10 +50,10 @@
       <xacro:thruster_volume thruster="heave_stbd_fwd" />
       <xacro:thruster_volume thruster="heave_port_aft" />
-      <xacro:thruster_volume thruster="heave_stbd_aft" /> -->
+      <xacro:thruster_volume thruster="heave_stbd_aft" />
     </plugin>
   </gazebo>
-    <!--             -->
+    <!--               -->
     <!-- Gazebo Colors -->
-    <!--             -->
+    <!--               -->
     <gazebo reference="housing_link">
       <material>Gazebo/Grey</material>
