Commit message: Cobbled together description from poor source data.

File: riptide_description/urdf/riptide.urdf.xacro (robot description, xacro)
@@ -17,17 +17,4 @@
                izz="1.9057706"/>
     </inertial>
-    <visual>
-      <origin xyz="0 0 0" rpy="0 ${M_PI/2} 0"/>
-      <geometry>
-        <cylinder radius="0.4" length="1.0"/>
-      </geometry>
-      <material name="Grey"/>
-    </visual>
-    <collision>
-      <origin xyz="0 0 0" rpy="0 ${M_PI/2} 0"/>
-      <geometry>
-        <cylinder radius="0.0483" length="0.1127"/>
-      </geometry>
-    </collision>
   </link>
   <joint name="base_frame" type="fixed">
@@ -38,10 +25,33 @@
   <link name="frame_link">
     <visual>
-      <origin xyz="0 0 0" rpy="0 0 0"/>
+      <origin xyz="0 -0.0483 0.08" rpy="${M_PI/2} 0 ${M_PI/2}"/>
       <geometry>
-        <box size="1.0 0.4 0.3"/>
+        <mesh filename="package://riptide_description/meshes/chassis.stl"/>
       </geometry>
-      <material name="Black"/>
+      <material name="frame"/>
     </visual>
   </link>
+  <joint name="base_housing" type="fixed">
+    <origin xyz="0 0 0" rpy="0 0 0"/>
+    <parent link="base_link"/>
+    <child link="housing_link"/>
+  </joint>
+  <link name="housing_link">
+    <visual>
+      <origin xyz="0 -0.0483 0.08" rpy="${M_PI/2} 0 ${M_PI/2}"/>
+      <geometry>
+        <mesh filename="package://riptide_description/meshes/main_housing.stl"/>
+      </geometry>
+      <material name="housing"/>
+    </visual>
+  </link>
+  <material name="frame">
+  <color rgba="0 0 0 1.0"/>
+  </material>
+  <material name="housing">
+  <color rgba="0.2 0.2 0.2 1.0"/>
+  </material>
+  <material name="thruster">
+    <color rgba="0.365 0 0 1.0"/>
+  </material>
 </robot>

File: riptide_description/urdf/t200_thrusters.urdf.xacro (robot description, xacro)
@@ -29,7 +29,7 @@
         <origin xyz="0 0 0" rpy="0 0 0" />
         <geometry>
-          <cylinder radius="0.0483" length="0.1127"/>
+          <mesh filename="package://riptide_description/meshes/t200.stl"/>
         </geometry>
-        <material name="Red"/>
+        <material name="thruster"/>
       </visual>
       <collision>

Commit message: Update physical properties.

File: riptide_description/urdf/riptide.urdf.xacro (robot description, xacro)
@@ -12,12 +12,12 @@
     <inertial>
       <origin xyz="0.00043180 0.03202940 -0.13947140" rpy="0 0 0"/>
-      <mass value="48.84278656"/>
-      <inertia ixx="0.55649783" ixy="0.00000000" ixz="0.00000000"
-               iyy="1.89075467" iyz="0.00000000"
-               izz="1.9057706"/>
+      <mass value="34.47940950"/>
+      <inertia ixx="0.50862680" ixy="-0.00114566" ixz="-0.03874012"
+               iyy="1.70892348" iyz="-0.00286748"
+               izz="1.77586420"/>
     </inertial>
   </link>
   <joint name="base_frame" type="fixed">
-    <origin xyz="0 0 0" rpy="0 0 0"/>
+    <origin xyz="0.1354 0.0003 0.0436" rpy="0 0 0"/>
     <parent link="base_link"/>
     <child link="frame_link"/>
@@ -32,7 +32,7 @@
     </visual>
   </link>
-  <joint name="base_housing" type="fixed">
+  <joint name="frame_housing" type="fixed">
     <origin xyz="0 0 0" rpy="0 0 0"/>
-    <parent link="base_link"/>
+    <parent link="frame_link"/>
     <child link="housing_link"/>
   </joint>

File: riptide_description/urdf/t200_thrusters.urdf.xacro (robot description, xacro)
@@ -4,14 +4,14 @@
 <!--                               -->
 <robot xmlns:xacro="http://ros.org/wiki/xacro">
-  <xacro:property name="sph_pos" value="-0.2128 0.1823 0.1384"/>
-  <xacro:property name="ssh_pos" value="-0.2128 -0.1823 0.1384"/>
-  <xacro:property name="spl_pos" value="-0.2128 0.1823 -0.0762"/>
-  <xacro:property name="ssl_pos" value="-0.2128 -0.1823 -0.0762"/>
-  <xacro:property name="sf_pos" value="0.3776 0.0110 -0.0838"/>
-  <xacro:property name="sa_pos" value="-0.3744 0.0110 -0.0838"/>
-  <xacro:property name="hpf_pos" value="0.2824 0.1823 0.007"/>
-  <xacro:property name="hsf_pos" value="0.2824 -0.1823 0.007"/>
-  <xacro:property name="hpa_pos" value="-0.2724 0.1823 0.0077"/>
-  <xacro:property name="hsa_pos" value="-0.2724 -0.1823 0.0077"/>
+  <xacro:property name="sph_pos" value="-0.2794 0.1824 0.0635"/>
+  <xacro:property name="ssh_pos" value="-0.2794 -0.1824 0.0635"/>
+  <xacro:property name="spl_pos" value="-0.2794 0.1824 -0.1588"/>
+  <xacro:property name="ssl_pos" value="-0.2794 -0.1824 -0.1588"/>
+  <xacro:property name="sf_pos" value="0.3220 0.0000 -0.1588"/>
+  <xacro:property name="sa_pos" value="-0.4300 0.0000 -0.1588"/>
+  <xacro:property name="hpf_pos" value="0.2268 0.1824 0.00782"/>
+  <xacro:property name="hsf_pos" value="0.2268 -0.1824 0.00782"/>
+  <xacro:property name="hpa_pos" value="-0.3279 0.1824 0.00782"/>
+  <xacro:property name="hsa_pos" value="-0.3279 -0.1824 0.00782"/>
   <xacro:macro name="t200_thruster" params="name position orientation">
     <link name="${name}_thruster">

Commit message: Add imu to description.

File: riptide_description/urdf/riptide.urdf.xacro (robot description, xacro)
@@ -46,4 +46,11 @@
     </visual>
   </link>
+  <joint name="base_imu" type="fixed">
+    <origin xyz="0 0 0" rpy="${M_PI} 0 0"/>
+    <parent link="base_link"/>
+    <child link="imu"/>
+  </joint>
+  <link name="imu">
+  </link>
   <material name="frame">
   <color rgba="0 0 0 1.0"/>

Commit message: Switch to new meshes.

File: riptide_description/urdf/riptide.urdf.xacro (robot description, xacro)
@@ -18,28 +18,84 @@
     </inertial>
   </link>
-  <joint name="base_frame" type="fixed">
-    <origin xyz="0.1354 0.0003 0.0436" rpy="0 0 0"/>
+  <joint name="base_housing" type="fixed">
+    <origin xyz="0 0 0" rpy="0 0 0"/>
     <parent link="base_link"/>
-    <child link="frame_link"/>
-  </joint>
-  <link name="frame_link">
-    <visual>
-      <origin xyz="0 -0.0483 0.08" rpy="${M_PI/2} 0 ${M_PI/2}"/>
-      <geometry>
-        <mesh filename="package://riptide_description/meshes/chassis.stl"/>
-      </geometry>
-      <material name="frame"/>
-    </visual>
-  </link>
-  <joint name="frame_housing" type="fixed">
-    <origin xyz="0 0 0" rpy="0 0 0"/>
-    <parent link="frame_link"/>
     <child link="housing_link"/>
   </joint>
   <link name="housing_link">
     <visual>
-      <origin xyz="0 -0.0483 0.08" rpy="${M_PI/2} 0 ${M_PI/2}"/>
+      <origin xyz="0 0 0" rpy="0 0 0"/>
       <geometry>
-        <mesh filename="package://riptide_description/meshes/main_housing.stl"/>
+        <mesh filename="package://riptide_description/meshes/riptide_housing.stl"/>
+      </geometry>
+      <material name="housing"/>
+    </visual>
+  </link>
+  <joint name="housing_chassis" type="fixed">
+    <origin xyz="-0.0556 0 -0.0749" rpy="0 0 0"/>
+    <parent link="housing_link"/>
+    <child link="chassis_link"/>
+  </joint>
+  <link name="chassis_link">
+    <visual>
+      <origin xyz="0 0 0" rpy="0 0 0"/>
+      <geometry>
+        <mesh filename="package://riptide_description/meshes/riptide_chassis.stl"/>
+      </geometry>
+      <material name="chassis"/>
+    </visual>
+  </link>
+  <joint name="chassis_acoustics" type="fixed">
+    <origin xyz="0.1699 0 -0.0584" rpy="0 0 0"/>
+    <parent link="chassis_link"/>
+    <child link="acoustic_link"/>
+  </joint>
+  <link name="acoustic_link">
+    <visual>
+      <origin xyz="0 0 0" rpy="0 0 0"/>
+      <geometry>
+        <mesh filename="package://riptide_description/meshes/riptide_acoustics.stl"/>
+      </geometry>
+      <material name="housing"/>
+    </visual>
+  </link>
+  <joint name="chassis_pneumatics" type="fixed">
+    <origin xyz="-0.1172 0 -0.0584" rpy="0 0 0"/>
+    <parent link="chassis_link"/>
+    <child link="pneumatic_link"/>
+  </joint>
+  <link name="pneumatic_link">
+    <visual>
+      <origin xyz="0 0 0" rpy="0 0 0"/>
+      <geometry>
+        <mesh filename="package://riptide_description/meshes/riptide_pneumatics.stl"/>
+      </geometry>
+      <material name="housing"/>
+    </visual>
+  </link>
+  <joint name="chassis_bat_port" type="fixed">
+    <origin xyz="-0.1781 0.1302 -0.0140" rpy="0 0 0"/>
+    <parent link="chassis_link"/>
+    <child link="bat_port_link"/>
+  </joint>
+  <link name="bat_port_link">
+    <visual>
+      <origin xyz="0 0 0" rpy="0 0 0"/>
+      <geometry>
+        <mesh filename="package://riptide_description/meshes/riptide_port_battery.stl"/>
+      </geometry>
+      <material name="housing"/>
+    </visual>
+  </link>
+  <joint name="chassis_bat_stbd" type="fixed">
+    <origin xyz="-0.1781 -0.1302 -0.0140" rpy="0 0 0"/>
+    <parent link="chassis_link"/>
+    <child link="bat_stbd_link"/>
+  </joint>
+  <link name="bat_stbd_link">
+    <visual>
+      <origin xyz="0 0 0" rpy="0 0 0"/>
+      <geometry>
+        <mesh filename="package://riptide_description/meshes/riptide_stbd_battery.stl"/>
       </geometry>
       <material name="housing"/>
@@ -53,5 +109,5 @@
   <link name="imu">
   </link>
-  <material name="frame">
+  <material name="chassis">
   <color rgba="0 0 0 1.0"/>
   </material>

File: riptide_description/urdf/t200_joints.urdf.xacro (robot description, xacro)
@@ -22,5 +22,5 @@
     <joint name="${name}_thruster_joint" type="fixed">
       <origin xyz="${position}" rpy="${orientation}"/>
-      <parent link="frame"/>
+      <parent link="chassis"/>
       <child link="${name}_thruster"/>
     </joint>

File: riptide_description/urdf/t200_thrusters.urdf.xacro (robot description, xacro)
@@ -4,14 +4,14 @@
 <!--                               -->
 <robot xmlns:xacro="http://ros.org/wiki/xacro">
-  <xacro:property name="sph_pos" value="-0.2794 0.1824 0.0635"/>
-  <xacro:property name="ssh_pos" value="-0.2794 -0.1824 0.0635"/>
-  <xacro:property name="spl_pos" value="-0.2794 0.1824 -0.1588"/>
-  <xacro:property name="ssl_pos" value="-0.2794 -0.1824 -0.1588"/>
-  <xacro:property name="sf_pos" value="0.3220 0.0000 -0.1588"/>
-  <xacro:property name="sa_pos" value="-0.4300 0.0000 -0.1588"/>
-  <xacro:property name="hpf_pos" value="0.2268 0.1824 0.00782"/>
-  <xacro:property name="hsf_pos" value="0.2268 -0.1824 0.00782"/>
-  <xacro:property name="hpa_pos" value="-0.3279 0.1824 0.00782"/>
-  <xacro:property name="hsa_pos" value="-0.3279 -0.1824 0.00782"/>
+  <xacro:property name="sph_pos" value="-0.2238 0.1824 0.1384"/>
+  <xacro:property name="ssh_pos" value="-0.2238 -0.1824 0.1384"/>
+  <xacro:property name="spl_pos" value="-0.2238 0.1824 -0.0838"/>
+  <xacro:property name="ssl_pos" value="-0.2238 -0.1824 -0.0838"/>
+  <xacro:property name="sf_pos" value="0.3776 0.0000 -0.0838"/>
+  <xacro:property name="sa_pos" value="-0.3744 0.0000 -0.0838"/>
+  <xacro:property name="hpf_pos" value="0.2824 0.1824 -0.0033"/>
+  <xacro:property name="hsf_pos" value="0.2824 -0.1824 -0.0033"/>
+  <xacro:property name="hpa_pos" value="-0.2724 0.1824 -0.0033"/>
+  <xacro:property name="hsa_pos" value="-0.2724 -0.1824 -0.0033"/>
   <xacro:macro name="t200_thruster" params="name position orientation">
     <link name="${name}_thruster">
@@ -26,5 +26,5 @@
         <origin xyz="0 0 0" rpy="0 0 0" />
         <geometry>
-          <mesh filename="package://riptide_description/meshes/t200.stl"/>
+          <mesh filename="package://riptide_description/meshes/blue_robotics_t200.stl"/>
         </geometry>
         <material name="thruster"/>
@@ -39,17 +39,17 @@
     <joint name="${name}_thruster_joint" type="fixed">
       <origin xyz="${position}" rpy="${orientation}"/>
-      <parent link="frame_link"/>
+      <parent link="chassis_link"/>
       <child link="${name}_thruster"/>
     </joint>
   </xacro:macro>
-  <xacro:t200_thruster name="surge_port_hi" position="${sph_pos}" orientation="0 ${M_PI/2} 0"/>
+  <xacro:t200_thruster name="surge_port_hi" position="${sph_pos}" orientation="0 ${-M_PI/2} ${M_PI}"/>
   <xacro:t200_thruster name="surge_stbd_hi" position="${ssh_pos}" orientation="0 ${M_PI/2} 0"/>
-  <xacro:t200_thruster name="surge_port_lo" position="${spl_pos}" orientation="0 ${M_PI/2} 0"/>
+  <xacro:t200_thruster name="surge_port_lo" position="${spl_pos}" orientation="0 ${-M_PI/2} ${M_PI}"/>
   <xacro:t200_thruster name="surge_stbd_lo" position="${ssl_pos}" orientation="0 ${M_PI/2} 0"/>
-  <xacro:t200_thruster name="sway_fwd" position="${sf_pos}" orientation="${3*M_PI/2} 0 0"/>
-  <xacro:t200_thruster name="sway_aft" position="${sa_pos}" orientation="${3*M_PI/2} 0 0"/>
-  <xacro:t200_thruster name="heave_port_fwd" position="${hpf_pos}" orientation="0 0 0"/>
+  <xacro:t200_thruster name="sway_fwd" position="${sf_pos}" orientation="0 ${M_PI/2} ${M_PI/2}"/>
+  <xacro:t200_thruster name="sway_aft" position="${sa_pos}" orientation="0 ${-M_PI/2} ${-M_PI/2}"/>
+  <xacro:t200_thruster name="heave_port_fwd" position="${hpf_pos}" orientation="0 0 ${M_PI}"/>
   <xacro:t200_thruster name="heave_stbd_fwd" position="${hsf_pos}" orientation="0 0 0"/>
-  <xacro:t200_thruster name="heave_port_aft" position="${hpa_pos}" orientation="0 0 0"/>
+  <xacro:t200_thruster name="heave_port_aft" position="${hpa_pos}" orientation="0 0 ${M_PI}"/>
   <xacro:t200_thruster name="heave_stbd_aft" position="${hsa_pos}" orientation="0 0 0"/>
 </robot>

Commit message: Starting Gazebo.

File: riptide_description/urdf/riptide.urdf.xacro (robot description, xacro)
@@ -11,8 +11,12 @@
   <xacro:include filename="riptide_links.urdf.xacro" />
   <xacro:include filename="riptide_joints.urdf.xacro" />
-  <material name="housing">
+  <xacro:include filename="riptide_sim.gazebo.xacro" />
+  <!--             -->
+  <!-- RVIZ Colors -->
+  <!--             -->
+  <material name="Grey">
     <color rgba="0.36 0.24 0.24 1.0"/>
   </material>
-  <material name="chassis">
+  <material name="FlatBlack">
     <color rgba="0.06 0.06 0.06 1.0"/>
   </material>

File: riptide_description/urdf/riptide_links.urdf.xacro (robot description, xacro)
@@ -16,5 +16,5 @@
         <mesh filename="${housing_mesh}" />
       </geometry>
-      <material name="housing" />
+      <material name="Grey" />
     </visual>
     <collision>
@@ -34,5 +34,5 @@
         <mesh filename="${chassis_mesh}" />
       </geometry>
-      <material name="chassis" />
+      <material name="FlatBlack" />
     </visual>
     <collision>

Commit message: Slightly positively buoyant.

File: riptide_description/urdf/riptide.urdf.xacro (robot description, xacro)
@@ -16,20 +16,14 @@
   <!--             -->
   <material name="Grey">
-    <color rgba="0.36 0.24 0.24 1.0"/>
+    <color rgba="0.5 0.5 0.5 1.0"/>
   </material>
   <material name="FlatBlack">
-    <color rgba="0.06 0.06 0.06 1.0"/>
+    <color rgba="0.1 0.1 0.1 1.0"/>
   </material>
-  <material name="acoustics">
-    <color rgba="0.12 0.12 0.12 1.0"/>
+  <material name="DarkGrey">
+    <color rgba="0.175 0.175 0.175 1.0"/>
   </material>
-  <material name="pneumatics">
-    <color rgba="0.12 0.12 0.12 1.0"/>
-  </material>
-  <material name="battery">
-    <color rgba="0.12 0.12 0.12 1.0"/>
-  </material>
-  <material name="thruster">
-    <color rgba="0.36 0.36 0.36 1.0"/>
+  <material name="RedBright">
+    <color rgba="0.87 0.26 0.07 1.0"/>
   </material>
 </robot>

File: riptide_description/urdf/riptide_joints.urdf.xacro (robot description, xacro)
@@ -1,7 +1,7 @@
 <?xml version="1.0"?>
 <robot xmlns:xacro="http://ros.org/wiki/xacro">
-  <!--                -->
-  <!-- Housing Joints -->
-  <!--                -->
+  <!--                   -->
+  <!-- Structural Joints -->
+  <!--                   -->
   <joint name="base_housing_joint" type="fixed">
     <origin xyz="${base_housing}" rpy="0 0 0"/>

File: riptide_description/urdf/riptide_links.urdf.xacro (robot description, xacro)
@@ -1,8 +1,12 @@
 <?xml version="1.0"?>
 <robot xmlns:xacro="http://ros.org/wiki/xacro">
-  <!--               -->
-  <!-- Housing Links -->
-  <!--               -->
+  <!--                  -->
+  <!-- Structural Links -->
+  <!--                  -->
   <link name="base_link">
+    <inertial>
+      <mass value="8.3901" />
+      <inertia ixx="0.0" ixy="0.0" ixz="0.0" iyy="0.0" iyz="0.0" izz="0.0" />
+    </inertial>
   </link>
   <link name="housing_link">
@@ -52,5 +56,5 @@
         <mesh filename="${acoustics_mesh}" />
       </geometry>
-      <material name="acoustics" />
+      <material name="DarkGrey" />
     </visual>
     <collision>
@@ -70,5 +74,5 @@
         <mesh filename="${pneumatics_mesh}" />
       </geometry>
-      <material name="pneumatics" />
+      <material name="DarkGrey" />
     </visual>
     <collision>
@@ -88,5 +92,5 @@
         <mesh filename="${port_battery_mesh}" />
       </geometry>
-      <material name="battery" />
+      <material name="DarkGrey" />
     </visual>
     <collision>
@@ -106,5 +110,5 @@
         <mesh filename="${stbd_battery_mesh}" />
       </geometry>
-        <material name="battery"/>
+        <material name="DarkGrey"/>
     </visual>
     <collision>
@@ -128,5 +132,5 @@
           <mesh filename="${thruster_mesh}" />
         </geometry>
-          <material name="thruster"/>
+          <material name="RedBright"/>
       </visual>
       <collision>

File: riptide_description/urdf/riptide_sim.gazebo.xacro (robot description, xacro)
@@ -5,9 +5,9 @@
     <!--                                -->
   <gazebo>
-    <!--  Buoyancy  -->
+    <!--  Buoyancy Plugin  -->
     <plugin name="BuoyancyPlugin" filename="libBuoyancyPlugin.so">
       <link name="base_link">
         <center_of_volume>0 0 0</center_of_volume>
-        <volume>0</volume>
+        <volume>0.0000000001</volume>
       </link>
       <link name="housing_link">
@@ -53,7 +53,7 @@
     </plugin>
   </gazebo>
-    <!--               -->
-    <!-- Gazebo Colors -->
-    <!--               -->
+    <!--                        -->
+    <!-- Gazebo Link Properties -->
+    <!--                        -->
     <gazebo reference="housing_link">
       <material>Gazebo/Grey</material>
@@ -62,3 +62,66 @@
       <material>Gazebo/FlatBlack</material>
     </gazebo>
+    <gazebo reference="acoustics_link">
+      <material>Gazebo/DarkGrey</material>
+    </gazebo>
+    <gazebo reference="pneumatics_link">
+      <material>Gazebo/DarkGrey</material>
+    </gazebo>
+    <gazebo reference="port_battery_link">
+      <material>Gazebo/DarkGrey</material>
+    </gazebo>
+    <gazebo reference="stbd_battery_link">
+      <material>Gazebo/DarkGrey</material>
+    </gazebo>
+    <xacro:macro name="thruster_link_gazebo" params="name">
+    <gazebo reference="${name}_link">
+      <material>Gazebo/RedBright</material>
+    </gazebo>
+    </xacro:macro>
+    <xacro:thruster_link_gazebo name="surge_port_hi" />
+    <xacro:thruster_link_gazebo name="surge_stbd_hi" />
+    <xacro:thruster_link_gazebo name="surge_port_lo" />
+    <xacro:thruster_link_gazebo name="surge_stbd_lo" />
+    <xacro:thruster_link_gazebo name="sway_fwd" />
+    <xacro:thruster_link_gazebo name="sway_aft" />
+    <xacro:thruster_link_gazebo name="heave_port_fwd" />
+    <xacro:thruster_link_gazebo name="heave_stbd_fwd" />
+    <xacro:thruster_link_gazebo name="heave_port_aft" />
+    <xacro:thruster_link_gazebo name="heave_stbd_aft" />
+    <!--                         -->
+    <!-- Gazebo Joint Properties -->
+    <!--                         -->
+    <gazebo reference="base_housing_joint">
+      <disableFixedJointLumping>true</disableFixedJointLumping>
+    </gazebo>
+    <gazebo reference="housing_chassis_joint">
+      <disableFixedJointLumping>true</disableFixedJointLumping>
+    </gazebo>
+    <gazebo reference="chassis_acoustics_joint">
+      <disableFixedJointLumping>true</disableFixedJointLumping>
+    </gazebo>
+    <gazebo reference="chassis_pneumatics_joint">
+      <disableFixedJointLumping>true</disableFixedJointLumping>
+    </gazebo>
+    <gazebo reference="chassis_port_battery_joint">
+      <disableFixedJointLumping>true</disableFixedJointLumping>
+    </gazebo>
+    <gazebo reference="chassis_stbd_battery_joint">
+      <disableFixedJointLumping>true</disableFixedJointLumping>
+    </gazebo>
+    <xacro:macro name="thruster_joint_gazebo" params="name">
+    <gazebo reference="${name}_joint">
+      <disableFixedJointLumping>true</disableFixedJointLumping>
+    </gazebo>
+    </xacro:macro>
+    <xacro:thruster_joint_gazebo name="surge_port_hi" />
+    <xacro:thruster_joint_gazebo name="surge_stbd_hi" />
+    <xacro:thruster_joint_gazebo name="surge_port_lo" />
+    <xacro:thruster_joint_gazebo name="surge_stbd_lo" />
+    <xacro:thruster_joint_gazebo name="sway_fwd" />
+    <xacro:thruster_joint_gazebo name="sway_aft" />
+    <xacro:thruster_joint_gazebo name="heave_port_fwd" />
+    <xacro:thruster_joint_gazebo name="heave_stbd_fwd" />
+    <xacro:thruster_joint_gazebo name="heave_port_aft" />
+    <xacro:thruster_joint_gazebo name="heave_stbd_aft" />
 </robot>
