Commit message: Cleanup hardware before adding sensors.

File: riptide_description/urdf/riptide.xacro (robot description, xacro)
@@ -15,15 +15,15 @@
   <!-- RVIZ Colors -->
   <!--             -->
+  <material name="RedBright">
+    <color rgba="0.87 0.26 0.07 1.0"/>
+  </material>
   <material name="Grey">
     <color rgba="0.5 0.5 0.5 1.0"/>
+  </material>
+  <material name="DarkGrey">
+    <color rgba="0.175 0.175 0.175 1.0"/>
   </material>
   <material name="FlatBlack">
     <color rgba="0.1 0.1 0.1 1.0"/>
   </material>
-  <material name="DarkGrey">
-    <color rgba="0.175 0.175 0.175 1.0"/>
-  </material>
-  <material name="RedBright">
-    <color rgba="0.87 0.26 0.07 1.0"/>
-  </material>
 </robot>

File: riptide_description/urdf/riptide_joints.xacro (robot description, xacro)
@@ -1,7 +1,7 @@
 <?xml version="1.0"?>
 <robot xmlns:xacro="http://ros.org/wiki/xacro">
-  <!--                   -->
-  <!-- Structural Joints -->
-  <!--                   -->
+  <!--                              -->
+  <!--        Riptide Joints        -->
+  <!--                              -->
   <joint name="base_housing_joint" type="fixed">
     <origin xyz="${base_housing}" rpy="0 0 0"/>
@@ -9,4 +9,7 @@
     <child link="housing_link"/>
   </joint>
+  <!--                -->
+  <!-- Housing Joints -->
+  <!--                -->
   <joint name="housing_chassis_joint" type="fixed">
     <origin xyz="${housing_chassis}" rpy="0 0 0"/>

File: riptide_description/urdf/riptide_links.xacro (robot description, xacro)
@@ -1,7 +1,7 @@
 <?xml version="1.0"?>
 <robot xmlns:xacro="http://ros.org/wiki/xacro">
-  <!--                  -->
-  <!-- Structural Links -->
-  <!--                  -->
+  <!--                             -->
+  <!--        Riptide Links        -->
+  <!--                             -->
   <link name="base_link">
     <inertial>
@@ -10,4 +10,7 @@
     </inertial>
   </link>
+  <!--               -->
+  <!-- Housing Links -->
+  <!--               -->
   <link name="housing_link">
     <inertial>

File: riptide_description/urdf/riptide_simulation.xacro (robot description, xacro)
@@ -1,9 +1,11 @@
 <?xml version="1.0"?>
 <robot name="riptide" xmlns:xacro="http://ros.org/wiki/xacro">
-    <!--                                -->
-    <!--  Gazebo Simulation Properties  -->
-    <!--                                -->
+    <!--                                 -->
+    <!--  Riptide Simulation Properties  -->
+    <!--                                 -->
   <gazebo>
-    <!--  Buoyancy Plugin  -->
+    <!--                                    -->
+    <!-- Gazebo Riptide Buoyancy Properties -->
+    <!--                                    -->
     <plugin name="BuoyancyPlugin" filename="libBuoyancyPlugin.so">
       <link name="base_link">
@@ -53,7 +55,7 @@
     </plugin>
   </gazebo>
-    <!--                        -->
-    <!-- Gazebo Link Properties -->
-    <!--                        -->
+    <!--                                -->
+    <!-- Gazebo Riptide Link Properties -->
+    <!--                                -->
     <gazebo reference="housing_link">
       <material>Gazebo/Grey</material>
@@ -89,7 +91,7 @@
     <xacro:thruster_link_gazebo name="heave_port_aft" />
     <xacro:thruster_link_gazebo name="heave_stbd_aft" />
-    <!--                         -->
-    <!-- Gazebo Joint Properties -->
-    <!--                         -->
+    <!--                                 -->
+    <!-- Gazebo Riptide Joint Properties -->
+    <!--                                 -->
     <gazebo reference="base_housing_joint">
       <disableFixedJointLumping>true</disableFixedJointLumping>

Commit message: Added forward stereo pair and removed some Xacro warnings

File: riptide_description/urdf/riptide.xacro (robot description, xacro)
@@ -8,8 +8,8 @@
 <robot name="riptide" xmlns:xacro="http://ros.org/wiki/xacro">
   <xacro:property name="M_PI" value="3.14159266"/>
-  <xacro:include filename="riptide_joints.xacro" />
-  <xacro:include filename="riptide_links.xacro" />
   <xacro:include filename="riptide_properties.xacro" />
   <xacro:include filename="riptide_simulation.xacro" />
+  <xacro:include filename="riptide_links.xacro" />
+  <xacro:include filename="riptide_joints.xacro" />
   <!--             -->
   <!-- RVIZ Colors -->

File: riptide_description/urdf/riptide_joints.xacro (robot description, xacro)
@@ -16,4 +16,24 @@
     <parent link="housing_link"/>
     <child link="imu_one_link"/>
+  </joint>
+  <joint name="housing_camera_fwd_port_joint" type="fixed">
+    <origin xyz="${housing_camera_fwd_port}" rpy="0 0 0" />
+    <parent link="housing_link"/>
+    <child link="camera_fwd_port_link"/>
+  </joint>
+  <joint name="housing_camera_fwd_stbd_joint" type="fixed">
+    <origin xyz="${housing_camera_fwd_stbd}" rpy="0 0 0" />
+    <parent link="housing_link"/>
+    <child link="camera_fwd_stbd_link"/>
+  </joint>
+  <joint name="housing_camera_down_port_joint" type="fixed">
+    <origin xyz="${housing_camera_down_port}" rpy="0 0 0" />
+    <parent link="housing_link"/>
+    <child link="camera_down_port_link"/>
+  </joint>
+  <joint name="housing_camera_down_stbd_joint" type="fixed">
+    <origin xyz="${housing_camera_down_stbd}" rpy="0 0 0" />
+    <parent link="housing_link"/>
+    <child link="camera_down_stbd_link"/>
   </joint>
   <!--                -->

File: riptide_description/urdf/riptide_links.xacro (robot description, xacro)
@@ -14,4 +14,28 @@
   <!--              -->
   <link name="imu_one_link">
+    <inertial>
+      <mass value="0.00001" />
+      <inertia ixx="0.0" ixy="0.0" ixz="0.0" iyy="0.0" iyz="0.0" izz="0.0" />
+    </inertial>
+  </link>
+  <link name="camera_fwd_port_link">
+    <inertial>
+      <mass value="0.00001" />
+      <inertia ixx="0.0" ixy="0.0" ixz="0.0" iyy="0.0" iyz="0.0" izz="0.0" />
+    </inertial>
+  </link>
+  <link name="camera_fwd_stbd_link">
+    <inertial>
+      <mass value="0.00001" />
+      <inertia ixx="0.0" ixy="0.0" ixz="0.0" iyy="0.0" iyz="0.0" izz="0.0" />
+    </inertial>
+  </link>
+  <link name="camera_down_port_link">
+    <inertial>
+      <mass value="0.00001" />
+      <inertia ixx="0.0" ixy="0.0" ixz="0.0" iyy="0.0" iyz="0.0" izz="0.0" />
+    </inertial>
+  </link>
+  <link name="camera_down_stbd_link">
     <inertial>
       <mass value="0.00001" />

File: riptide_description/urdf/riptide_properties.xacro (robot description, xacro)
@@ -1,7 +1,8 @@
 <?xml version="1.0"?>
 <robot xmlns:xacro="http://ros.org/wiki/xacro">
-  <xacro:property name="housing_camera_port" value="0.2744 0.0400 -0.0004" />
-  <xacro:property name="housing_camera_stbd" value="0.2744 -0.0400 -0.0004" />
-  <xacro:property name="housing_camera_down" value="0.2360 0.0000 -0.0620" />
+  <xacro:property name="housing_camera_fwd_port" value="0.4 0.0400 -0.0004" />
+  <xacro:property name="housing_camera_fwd_stbd" value="0.4 -0.0400 -0.0004" />
+  <xacro:property name="housing_camera_down_port" value="0.2360 0.0400 -0.0620" />
+  <xacro:property name="housing_camera_down_stbd" value="0.2360 -0.0400 -0.0620" />
   <xacro:property name="housing_depth_sensor" value="0.0000 0.0000 0.1049" />
   <xacro:property name="housing_imu_one" value="0.1322 -0.0056 0.0268" />

File: riptide_description/urdf/riptide_simulation.xacro (robot description, xacro)
@@ -1,7 +1,7 @@
 <?xml version="1.0"?>
 <robot name="riptide" xmlns:xacro="http://ros.org/wiki/xacro">
-    <!--                                 -->
-    <!--  Riptide Simulation Properties  -->
-    <!--                                 -->
+  <!--                                 -->
+  <!--  Riptide Simulation Properties  -->
+  <!--                                 -->
   <gazebo>
     <!--                                  -->
@@ -29,129 +29,199 @@
     <!-- Gazebo Riptide Buoyancy Properties -->
     <!--                                    -->
-    <plugin name="BuoyancyPlugin" filename="libBuoyancyPlugin.so">
-      <link name="imu_one_link">
-        <center_of_volume>0 0 0</center_of_volume>
-        <volume>0.0000000001</volume>
-      </link>
-      <link name="base_link">
-        <center_of_volume>0 0 0</center_of_volume>
-        <volume>0.0000000001</volume>
-      </link>
-      <link name="housing_link">
-        <center_of_volume>${housing_cov}</center_of_volume>
-        <volume>${housing_volume}</volume>
-      </link>
-      <link name="chassis_link">
-        <center_of_volume>${chassis_cov}</center_of_volume>
-        <volume>${chassis_volume}</volume>
-      </link>
-      <link name="acoustics_link">
-        <center_of_volume>${acoustics_cov}</center_of_volume>
-        <volume>${acoustics_volume}</volume>
-      </link>
-      <link name="pneumatics_link">
-        <center_of_volume>${pneumatics_cov}</center_of_volume>
-        <volume>${pneumatics_volume}</volume>
-      </link>
-      <link name="port_battery_link">
-        <center_of_volume>${port_battery_cov}</center_of_volume>
-        <volume>${port_battery_volume}</volume>
-      </link>
-      <link name="stbd_battery_link">
-        <center_of_volume>${stbd_battery_cov}</center_of_volume>
-        <volume>${stbd_battery_volume}</volume>
-      </link>
-      <xacro:macro name="thruster_volume" params="thruster">
-        <link name="${thruster}_link">
-          <center_of_volume>${thruster_cov}</center_of_volume>
-          <volume>${thruster_volume}</volume>
-        </link>
-      </xacro:macro>
-      <xacro:thruster_volume thruster="surge_port_hi" />
-      <xacro:thruster_volume thruster="surge_stbd_hi" />
-      <xacro:thruster_volume thruster="surge_port_lo" />
-      <xacro:thruster_volume thruster="surge_stbd_lo" />
-      <xacro:thruster_volume thruster="sway_fwd" />
-      <xacro:thruster_volume thruster="sway_aft" />
-      <xacro:thruster_volume thruster="heave_port_fwd" />
-      <xacro:thruster_volume thruster="heave_stbd_fwd" />
-      <xacro:thruster_volume thruster="heave_port_aft" />
-      <xacro:thruster_volume thruster="heave_stbd_aft" />
+    <!-- <plugin name="BuoyancyPlugin" filename="libBuoyancyPlugin.so">
+    <link name="imu_one_link">
+    <center_of_volume>0 0 0</center_of_volume>
+    <volume>0.0000000001</volume>
+  </link>
+  <link name="base_link">
+  <center_of_volume>0 0 0</center_of_volume>
+  <volume>0.0000000001</volume>
+</link>
+<link name="housing_link">
+<center_of_volume>${housing_cov}</center_of_volume>
+<volume>${housing_volume}</volume>
+</link>
+<link name="chassis_link">
+<center_of_volume>${chassis_cov}</center_of_volume>
+<volume>${chassis_volume}</volume>
+</link>
+<link name="acoustics_link">
+<center_of_volume>${acoustics_cov}</center_of_volume>
+<volume>${acoustics_volume}</volume>
+</link>
+<link name="pneumatics_link">
+<center_of_volume>${pneumatics_cov}</center_of_volume>
+<volume>${pneumatics_volume}</volume>
+</link>
+<link name="port_battery_link">
+<center_of_volume>${port_battery_cov}</center_of_volume>
+<volume>${port_battery_volume}</volume>
+</link>
+<link name="stbd_battery_link">
+<center_of_volume>${stbd_battery_cov}</center_of_volume>
+<volume>${stbd_battery_volume}</volume>
+</link>
+<xacro:macro name="thruster_volume" params="thruster">
+<link name="${thruster}_link">
+<center_of_volume>${thruster_cov}</center_of_volume>
+<volume>${thruster_volume}</volume>
+</link>
+</xacro:macro>
+<xacro:thruster_volume thruster="surge_port_hi" />
+<xacro:thruster_volume thruster="surge_stbd_hi" />
+<xacro:thruster_volume thruster="surge_port_lo" />
+<xacro:thruster_volume thruster="surge_stbd_lo" />
+<xacro:thruster_volume thruster="sway_fwd" />
+<xacro:thruster_volume thruster="sway_aft" />
+<xacro:thruster_volume thruster="heave_port_fwd" />
+<xacro:thruster_volume thruster="heave_stbd_fwd" />
+<xacro:thruster_volume thruster="heave_port_aft" />
+<xacro:thruster_volume thruster="heave_stbd_aft" />
+</plugin> -->
+</gazebo>
+<!--                                -->
+<!-- Gazebo Riptide Link Properties -->
+<!--                                -->
+<gazebo reference="housing_link">
+  <material>Gazebo/Grey</material>
+</gazebo>
+<gazebo reference="chassis_link">
+  <material>Gazebo/FlatBlack</material>
+</gazebo>
+<gazebo reference="acoustics_link">
+  <material>Gazebo/DarkGrey</material>
+</gazebo>
+<gazebo reference="pneumatics_link">
+  <material>Gazebo/DarkGrey</material>
+</gazebo>
+<gazebo reference="port_battery_link">
+  <material>Gazebo/DarkGrey</material>
+</gazebo>
+<gazebo reference="stbd_battery_link">
+  <material>Gazebo/DarkGrey</material>
+</gazebo>
+<xacro:macro name="thruster_link_gazebo" params="name">
+  <gazebo reference="${name}_link">
+    <material>Gazebo/RedBright</material>
+  </gazebo>
+</xacro:macro>
+<xacro:thruster_link_gazebo name="surge_port_hi" />
+<xacro:thruster_link_gazebo name="surge_stbd_hi" />
+<xacro:thruster_link_gazebo name="surge_port_lo" />
+<xacro:thruster_link_gazebo name="surge_stbd_lo" />
+<xacro:thruster_link_gazebo name="sway_fwd" />
+<xacro:thruster_link_gazebo name="sway_aft" />
+<xacro:thruster_link_gazebo name="heave_port_fwd" />
+<xacro:thruster_link_gazebo name="heave_stbd_fwd" />
+<xacro:thruster_link_gazebo name="heave_port_aft" />
+<xacro:thruster_link_gazebo name="heave_stbd_aft" />
+<!--                                 -->
+<!-- Gazebo Riptide Joint Properties -->
+<!--                                 -->
+<gazebo reference="housing_imu_one_joint">
+  <disableFixedJointLumping>true</disableFixedJointLumping>
+</gazebo>
+<gazebo reference="housing_camera_fwd_port_joint">
+  <disableFixedJointLumping>true</disableFixedJointLumping>
+</gazebo>
+<gazebo reference="housing_camera_fwd_stbd_joint">
+  <disableFixedJointLumping>true</disableFixedJointLumping>
+</gazebo>
+<gazebo reference="housing_camera_down_port_joint">
+  <disableFixedJointLumping>true</disableFixedJointLumping>
+</gazebo>
+<gazebo reference="housing_camera_down_stbd_joint">
+  <disableFixedJointLumping>true</disableFixedJointLumping>
+</gazebo>
+<gazebo reference="base_housing_joint">
+  <disableFixedJointLumping>true</disableFixedJointLumping>
+</gazebo>
+<gazebo reference="housing_chassis_joint">
+  <disableFixedJointLumping>true</disableFixedJointLumping>
+</gazebo>
+<gazebo reference="chassis_acoustics_joint">
+  <disableFixedJointLumping>true</disableFixedJointLumping>
+</gazebo>
+<gazebo reference="chassis_pneumatics_joint">
+  <disableFixedJointLumping>true</disableFixedJointLumping>
+</gazebo>
+<gazebo reference="chassis_port_battery_joint">
+  <disableFixedJointLumping>true</disableFixedJointLumping>
+</gazebo>
+<gazebo reference="chassis_stbd_battery_joint">
+  <disableFixedJointLumping>true</disableFixedJointLumping>
+</gazebo>
+<xacro:macro name="thruster_joint_gazebo" params="name">
+  <gazebo reference="${name}_joint">
+    <disableFixedJointLumping>true</disableFixedJointLumping>
+  </gazebo>
+</xacro:macro>
+<xacro:thruster_joint_gazebo name="surge_port_hi" />
+<xacro:thruster_joint_gazebo name="surge_stbd_hi" />
+<xacro:thruster_joint_gazebo name="surge_port_lo" />
+<xacro:thruster_joint_gazebo name="surge_stbd_lo" />
+<xacro:thruster_joint_gazebo name="sway_fwd" />
+<xacro:thruster_joint_gazebo name="sway_aft" />
+<xacro:thruster_joint_gazebo name="heave_port_fwd" />
+<xacro:thruster_joint_gazebo name="heave_stbd_fwd" />
+<xacro:thruster_joint_gazebo name="heave_port_aft" />
+<xacro:thruster_joint_gazebo name="heave_stbd_aft" />
+<!--                                  -->
+<!-- Gazebo Riptide Camera Properties -->
+<!--                                  -->
+<!-- Camera 1 -->
+<gazebo reference="camera_fwd_port_link">
+  <sensor type="multicamera" name="stereo_camera">
+    <update_rate>30.0</update_rate>
+    <camera name="left">
+      <horizontal_fov>1.3962634</horizontal_fov>
+      <image>
+        <width>800</width>
+        <height>800</height>
+        <format>R8G8B8</format>
+      </image>
+      <clip>
+        <near>0.02</near>
+        <far>300</far>
+      </clip>
+      <noise>
+        <type>gaussian</type>
+        <mean>0.0</mean>
+        <stddev>0.007</stddev>
+      </noise>
+    </camera>
+    <camera name="right">
+      <pose>0 -0.07 0 0 0 0</pose>
+      <horizontal_fov>1.3962634</horizontal_fov>
+      <image>
+        <width>800</width>
+        <height>800</height>
+        <format>R8G8B8</format>
+      </image>
+      <clip>
+        <near>0.02</near>
+        <far>300</far>
+      </clip>
+      <noise>
+        <type>gaussian</type>
+        <mean>0.0</mean>
+        <stddev>0.007</stddev>
+      </noise>
+    </camera>
+    <plugin name="stereo_camera_controller" filename="libgazebo_ros_multicamera.so">
+      <alwaysOn>true</alwaysOn>
+      <updateRate>0.0</updateRate>
+      <cameraName>riptide/stereo_fwd</cameraName>
+      <imageTopicName>image_raw</imageTopicName>
+      <cameraInfoTopicName>camera_info</cameraInfoTopicName>
+      <frameName>camera_fwd_port_link</frameName>
+      <hackBaseline>0.07</hackBaseline>
+      <distortionK1>0.0</distortionK1>
+      <distortionK2>0.0</distortionK2>
+      <distortionK3>0.0</distortionK3>
+      <distortionT1>0.0</distortionT1>
+      <distortionT2>0.0</distortionT2>
     </plugin>
-  </gazebo>
-    <!--                                -->
-    <!-- Gazebo Riptide Link Properties -->
-    <!--                                -->
-    <gazebo reference="housing_link">
-      <material>Gazebo/Grey</material>
-    </gazebo>
-    <gazebo reference="chassis_link">
-      <material>Gazebo/FlatBlack</material>
-    </gazebo>
-    <gazebo reference="acoustics_link">
-      <material>Gazebo/DarkGrey</material>
-    </gazebo>
-    <gazebo reference="pneumatics_link">
-      <material>Gazebo/DarkGrey</material>
-    </gazebo>
-    <gazebo reference="port_battery_link">
-      <material>Gazebo/DarkGrey</material>
-    </gazebo>
-    <gazebo reference="stbd_battery_link">
-      <material>Gazebo/DarkGrey</material>
-    </gazebo>
-    <xacro:macro name="thruster_link_gazebo" params="name">
-    <gazebo reference="${name}_link">
-      <material>Gazebo/RedBright</material>
-    </gazebo>
-    </xacro:macro>
-    <xacro:thruster_link_gazebo name="surge_port_hi" />
-    <xacro:thruster_link_gazebo name="surge_stbd_hi" />
-    <xacro:thruster_link_gazebo name="surge_port_lo" />
-    <xacro:thruster_link_gazebo name="surge_stbd_lo" />
-    <xacro:thruster_link_gazebo name="sway_fwd" />
-    <xacro:thruster_link_gazebo name="sway_aft" />
-    <xacro:thruster_link_gazebo name="heave_port_fwd" />
-    <xacro:thruster_link_gazebo name="heave_stbd_fwd" />
-    <xacro:thruster_link_gazebo name="heave_port_aft" />
-    <xacro:thruster_link_gazebo name="heave_stbd_aft" />
-    <!--                                 -->
-    <!-- Gazebo Riptide Joint Properties -->
-    <!--                                 -->
-    <gazebo reference="housing_imu_one_joint">
-      <disableFixedJointLumping>true</disableFixedJointLumping>
-    </gazebo>
-    <gazebo reference="base_housing_joint">
-      <disableFixedJointLumping>true</disableFixedJointLumping>
-    </gazebo>
-    <gazebo reference="housing_chassis_joint">
-      <disableFixedJointLumping>true</disableFixedJointLumping>
-    </gazebo>
-    <gazebo reference="chassis_acoustics_joint">
-      <disableFixedJointLumping>true</disableFixedJointLumping>
-    </gazebo>
-    <gazebo reference="chassis_pneumatics_joint">
-      <disableFixedJointLumping>true</disableFixedJointLumping>
-    </gazebo>
-    <gazebo reference="chassis_port_battery_joint">
-      <disableFixedJointLumping>true</disableFixedJointLumping>
-    </gazebo>
-    <gazebo reference="chassis_stbd_battery_joint">
-      <disableFixedJointLumping>true</disableFixedJointLumping>
-    </gazebo>
-    <xacro:macro name="thruster_joint_gazebo" params="name">
-    <gazebo reference="${name}_joint">
-      <disableFixedJointLumping>true</disableFixedJointLumping>
-    </gazebo>
-    </xacro:macro>
-    <xacro:thruster_joint_gazebo name="surge_port_hi" />
-    <xacro:thruster_joint_gazebo name="surge_stbd_hi" />
-    <xacro:thruster_joint_gazebo name="surge_port_lo" />
-    <xacro:thruster_joint_gazebo name="surge_stbd_lo" />
-    <xacro:thruster_joint_gazebo name="sway_fwd" />
-    <xacro:thruster_joint_gazebo name="sway_aft" />
-    <xacro:thruster_joint_gazebo name="heave_port_fwd" />
-    <xacro:thruster_joint_gazebo name="heave_stbd_fwd" />
-    <xacro:thruster_joint_gazebo name="heave_port_aft" />
-    <xacro:thruster_joint_gazebo name="heave_stbd_aft" />
+  </sensor>
+</gazebo>
 </robot>
