Commit message: Cured symptoms of potential bug with BuoyancyPlugin. Added collision geometries to sensors.

File: riptide_description/urdf/riptide.xacro (robot description, xacro)
@@ -9,6 +9,6 @@
   <xacro:property name="M_PI" value="3.14159266"/>
   <xacro:include filename="riptide_properties.xacro" />
+  <xacro:include filename="riptide_links.xacro" />
   <xacro:include filename="riptide_simulation.xacro" />
-  <xacro:include filename="riptide_links.xacro" />
   <xacro:include filename="riptide_joints.xacro" />
   <!--             -->

File: riptide_description/urdf/riptide_joints.xacro (robot description, xacro)
@@ -8,32 +8,4 @@
     <parent link="base_link"/>
     <child link="housing_link"/>
-  </joint>
-  <!--               -->
-  <!-- Sensor Joints -->
-  <!--               -->
-  <joint name="housing_imu_one_joint" type="fixed">
-    <origin xyz="${housing_imu_one}" rpy="0 0 0" />
-    <parent link="housing_link"/>
-    <child link="imu_one_link"/>
-  </joint>
-  <joint name="housing_camera_fwd_port_joint" type="fixed">
-    <origin xyz="${housing_camera_fwd_port}" rpy="0 0 0" />
-    <parent link="housing_link"/>
-    <child link="camera_fwd_port_link"/>
-  </joint>
-  <joint name="housing_camera_fwd_stbd_joint" type="fixed">
-    <origin xyz="${housing_camera_fwd_stbd}" rpy="0 0 0" />
-    <parent link="housing_link"/>
-    <child link="camera_fwd_stbd_link"/>
-  </joint>
-  <joint name="housing_camera_down_port_joint" type="fixed">
-    <origin xyz="${housing_camera_down_port}" rpy="0 0 0" />
-    <parent link="housing_link"/>
-    <child link="camera_down_port_link"/>
-  </joint>
-  <joint name="housing_camera_down_stbd_joint" type="fixed">
-    <origin xyz="${housing_camera_down_stbd}" rpy="0 0 0" />
-    <parent link="housing_link"/>
-    <child link="camera_down_stbd_link"/>
   </joint>
   <!--                -->
@@ -85,3 +57,31 @@
   <xacro:thruster_joint name="heave_port_aft" p="${chassis_heave_port_aft}" o="${align_heave_port_aft}"/>
   <xacro:thruster_joint name="heave_stbd_aft" p="${chassis_heave_stbd_aft}" o="${align_heave_stbd_aft}"/>
+    <!--               -->
+    <!-- Sensor Joints -->
+    <!--               -->
+    <joint name="housing_imu_one_joint" type="fixed">
+      <origin xyz="${housing_imu_one}" rpy="0 0 0" />
+      <parent link="housing_link"/>
+      <child link="imu_one_link"/>
+    </joint>
+    <joint name="housing_camera_fwd_port_joint" type="fixed">
+      <origin xyz="${housing_camera_fwd_port}" rpy="0 0 0" />
+      <parent link="housing_link"/>
+      <child link="camera_fwd_port_link"/>
+    </joint>
+    <joint name="housing_camera_fwd_stbd_joint" type="fixed">
+      <origin xyz="${housing_camera_fwd_stbd}" rpy="0 0 0" />
+      <parent link="housing_link"/>
+      <child link="camera_fwd_stbd_link"/>
+    </joint>
+    <joint name="housing_camera_down_port_joint" type="fixed">
+      <origin xyz="${housing_camera_down_port}" rpy="0 0 0" />
+      <parent link="housing_link"/>
+      <child link="camera_down_port_link"/>
+    </joint>
+    <joint name="housing_camera_down_stbd_joint" type="fixed">
+      <origin xyz="${housing_camera_down_stbd}" rpy="0 0 0" />
+      <parent link="housing_link"/>
+      <child link="camera_down_stbd_link"/>
+    </joint>
 </robot>

File: riptide_description/urdf/riptide_links.xacro (robot description, xacro)
@@ -6,37 +6,4 @@
   <link name="base_link">
     <inertial>
-      <mass value="8.3901" />
-      <inertia ixx="0.0" ixy="0.0" ixz="0.0" iyy="0.0" iyz="0.0" izz="0.0" />
-    </inertial>
-  </link>
-  <!--              -->
-  <!-- Sensor Links -->
-  <!--              -->
-  <link name="imu_one_link">
-    <inertial>
-      <mass value="0.00001" />
-      <inertia ixx="0.0" ixy="0.0" ixz="0.0" iyy="0.0" iyz="0.0" izz="0.0" />
-    </inertial>
-  </link>
-  <link name="camera_fwd_port_link">
-    <inertial>
-      <mass value="0.00001" />
-      <inertia ixx="0.0" ixy="0.0" ixz="0.0" iyy="0.0" iyz="0.0" izz="0.0" />
-    </inertial>
-  </link>
-  <link name="camera_fwd_stbd_link">
-    <inertial>
-      <mass value="0.00001" />
-      <inertia ixx="0.0" ixy="0.0" ixz="0.0" iyy="0.0" iyz="0.0" izz="0.0" />
-    </inertial>
-  </link>
-  <link name="camera_down_port_link">
-    <inertial>
-      <mass value="0.00001" />
-      <inertia ixx="0.0" ixy="0.0" ixz="0.0" iyy="0.0" iyz="0.0" izz="0.0" />
-    </inertial>
-  </link>
-  <link name="camera_down_stbd_link">
-    <inertial>
       <mass value="0.00001" />
       <inertia ixx="0.0" ixy="0.0" ixz="0.0" iyy="0.0" iyz="0.0" izz="0.0" />
@@ -153,5 +120,5 @@
       </geometry>
     </collision>
-  </link>
+  </link> -->
   <!--                -->
   <!-- Thruster Links -->
@@ -187,3 +154,66 @@
   <xacro:thruster_link thruster="heave_port_aft" />
   <xacro:thruster_link thruster="heave_stbd_aft" />
+  <!--              -->
+  <!-- Sensor Links -->
+  <!--              -->
+  <link name="imu_one_link">
+    <inertial>
+      <mass value="8" />
+      <inertia ixx="0.0" ixy="0.0" ixz="0.0" iyy="0.0" iyz="0.0" izz="0.0" />
+    </inertial>
+    <!-- Collision Geometry necessary for Buoyancy Plugin to work! -->
+    <collision>
+      <geometry>
+        <box size="0.0001 0.0001 0.0001" />
+      </geometry>
+    </collision>
+  </link>
+  <link name="camera_fwd_port_link">
+    <inertial>
+      <mass value="0.00001" />
+      <inertia ixx="0.0" ixy="0.0" ixz="0.0" iyy="0.0" iyz="0.0" izz="0.0" />
+    </inertial>
+    <!-- Collision Geometry necessary for Buoyancy Plugin to work! -->
+    <collision>
+      <geometry>
+        <box size="0.0001 0.0001 0.0001" />
+      </geometry>
+    </collision>
+  </link>
+  <link name="camera_fwd_stbd_link">
+    <inertial>
+      <mass value="0.00001" />
+      <inertia ixx="0.0" ixy="0.0" ixz="0.0" iyy="0.0" iyz="0.0" izz="0.0" />
+    </inertial>
+    <!-- Collision Geometry necessary for Buoyancy Plugin to work! -->
+    <collision>
+      <geometry>
+        <box size="0.0001 0.0001 0.0001" />
+      </geometry>
+    </collision>
+  </link>
+  <link name="camera_down_port_link">
+    <inertial>
+      <mass value="0.00001" />
+      <inertia ixx="0.0" ixy="0.0" ixz="0.0" iyy="0.0" iyz="0.0" izz="0.0" />
+    </inertial>
+    <!-- Collision Geometry necessary for Buoyancy Plugin to work! -->
+    <collision>
+      <geometry>
+        <box size="0.0001 0.0001 0.0001" />
+      </geometry>
+    </collision>
+  </link>
+  <link name="camera_down_stbd_link">
+    <inertial>
+      <mass value="0.00001" />
+      <inertia ixx="0.0" ixy="0.0" ixz="0.0" iyy="0.0" iyz="0.0" izz="0.0" />
+    </inertial>
+    <!-- Collision Geometry necessary for Buoyancy Plugin to work! -->
+    <collision>
+      <geometry>
+        <box size="0.0001 0.0001 0.0001" />
+      </geometry>
+    </collision>
+  </link>
 </robot>

File: riptide_description/urdf/riptide_simulation.xacro (robot description, xacro)
@@ -1,4 +1,91 @@
 <?xml version="1.0"?>
 <robot name="riptide" xmlns:xacro="http://ros.org/wiki/xacro">
+  <!--                                -->
+  <!-- Gazebo Riptide Link Properties -->
+  <!--                                -->
+  <gazebo reference="housing_link">
+    <material>Gazebo/Grey</material>
+  </gazebo>
+  <gazebo reference="chassis_link">
+    <material>Gazebo/FlatBlack</material>
+  </gazebo>
+  <gazebo reference="acoustics_link">
+    <material>Gazebo/DarkGrey</material>
+  </gazebo>
+  <gazebo reference="pneumatics_link">
+    <material>Gazebo/DarkGrey</material>
+  </gazebo>
+  <gazebo reference="port_battery_link">
+    <material>Gazebo/DarkGrey</material>
+  </gazebo>
+  <gazebo reference="stbd_battery_link">
+    <material>Gazebo/DarkGrey</material>
+  </gazebo>
+  <xacro:macro name="thruster_link_gazebo" params="name">
+    <gazebo reference="${name}_link">
+      <material>Gazebo/RedBright</material>
+    </gazebo>
+  </xacro:macro>
+  <xacro:thruster_link_gazebo name="surge_port_hi" />
+  <xacro:thruster_link_gazebo name="surge_stbd_hi" />
+  <xacro:thruster_link_gazebo name="surge_port_lo" />
+  <xacro:thruster_link_gazebo name="surge_stbd_lo" />
+  <xacro:thruster_link_gazebo name="sway_fwd" />
+  <xacro:thruster_link_gazebo name="sway_aft" />
+  <xacro:thruster_link_gazebo name="heave_port_fwd" />
+  <xacro:thruster_link_gazebo name="heave_stbd_fwd" />
+  <xacro:thruster_link_gazebo name="heave_port_aft" />
+  <xacro:thruster_link_gazebo name="heave_stbd_aft" />
+  <!--                                 -->
+  <!-- Gazebo Riptide Joint Properties -->
+  <!--                                 -->
+  <gazebo reference="base_housing_joint">
+    <disableFixedJointLumping>true</disableFixedJointLumping>
+  </gazebo>
+  <gazebo reference="housing_chassis_joint">
+    <disableFixedJointLumping>true</disableFixedJointLumping>
+  </gazebo>
+  <gazebo reference="chassis_acoustics_joint">
+    <disableFixedJointLumping>true</disableFixedJointLumping>
+  </gazebo>
+  <gazebo reference="chassis_pneumatics_joint">
+    <disableFixedJointLumping>true</disableFixedJointLumping>
+  </gazebo>
+  <gazebo reference="chassis_port_battery_joint">
+    <disableFixedJointLumping>true</disableFixedJointLumping>
+  </gazebo>
+  <gazebo reference="chassis_stbd_battery_joint">
+    <disableFixedJointLumping>true</disableFixedJointLumping>
+  </gazebo>
+  <xacro:macro name="thruster_joint_gazebo" params="name">
+    <gazebo reference="${name}_joint">
+      <disableFixedJointLumping>true</disableFixedJointLumping>
+    </gazebo>
+  </xacro:macro>
+  <xacro:thruster_joint_gazebo name="surge_port_hi" />
+  <xacro:thruster_joint_gazebo name="surge_stbd_hi" />
+  <xacro:thruster_joint_gazebo name="surge_port_lo" />
+  <xacro:thruster_joint_gazebo name="surge_stbd_lo" />
+  <xacro:thruster_joint_gazebo name="sway_fwd" />
+  <xacro:thruster_joint_gazebo name="sway_aft" />
+  <xacro:thruster_joint_gazebo name="heave_port_fwd" />
+  <xacro:thruster_joint_gazebo name="heave_stbd_fwd" />
+  <xacro:thruster_joint_gazebo name="heave_port_aft" />
+  <xacro:thruster_joint_gazebo name="heave_stbd_aft" /> -->
+    <gazebo reference="housing_imu_one_joint">
+      <disableFixedJointLumping>true</disableFixedJointLumping>
+    </gazebo>
+    <gazebo reference="housing_camera_fwd_port_joint">
+      <disableFixedJointLumping>true</disableFixedJointLumping>
+    </gazebo>
+    <gazebo reference="housing_camera_fwd_stbd_joint">
+      <disableFixedJointLumping>true</disableFixedJointLumping>
+    </gazebo>
+    <gazebo reference="housing_camera_down_port_joint">
+      <disableFixedJointLumping>true</disableFixedJointLumping>
+    </gazebo>
+    <gazebo reference="housing_camera_down_stbd_joint">
+      <disableFixedJointLumping>true</disableFixedJointLumping>
+    </gazebo>
   <!--                                 -->
   <!--  Riptide Simulation Properties  -->
@@ -8,4 +95,5 @@
     <!-- Gazebo Riptide Sensor Properties -->
     <!--                                  -->
+<!--
     <plugin name="imu_one" filename="libgazebo_ros_imu.so">
       <robotNamespace></robotNamespace>
@@ -18,12 +106,13 @@
       <updateRate>100.0</updateRate>
       <frameName>imu_one_link</frameName>
-    </plugin>
+    </plugin> -->
     <!--                                    -->
     <!-- Gazebo Riptide Thruster Properties -->
     <!--                                    -->
+<!--
     <plugin filename="libgazebo_ros_riptide_thrust.so" name="thrust">
       <robotNamespace></robotNamespace>
       <topicName>/command/thrust</topicName>
-    </plugin>
+    </plugin> -->
     <!--                                    -->
     <!-- Gazebo Riptide Buoyancy Properties -->
@@ -31,25 +120,5 @@
 <plugin name="BuoyancyPlugin" filename="libBuoyancyPlugin.so">
 <robotNamespace></robotNamespace>
-<fluid_density>1</fluid_density>
-<link name="imu_one_link">
-    <center_of_volume>0 0 0</center_of_volume>
-    <volume>0.000000001</volume>
-</link>
-<link name="camera_fwd_port_link">
-    <center_of_volume>0 0 0</center_of_volume>
-    <volume>0.000000001</volume>
-</link>
-<link name="camera_fwd_stbd_link">
-    <center_of_volume>0 0 0</center_of_volume>
-    <volume>0.000000001</volume>
-</link>
-<link name="camera_down_port_link">
-    <center_of_volume>0 0 0</center_of_volume>
-    <volume>0.000000001</volume>
-</link>
-<link name="camera_down_stbd_link">
-    <center_of_volume>0 0 0</center_of_volume>
-    <volume>0.000000001</volume>
-</link>
+<fluid_density>195</fluid_density>
 <link name="base_link">
   <center_of_volume>0 0 0</center_of_volume>
@@ -96,93 +165,26 @@
 <xacro:thruster_volume thruster="heave_port_aft" />
 <xacro:thruster_volume thruster="heave_stbd_aft" />
+<link name="imu_one_link">
+    <center_of_volume>0 0 0</center_of_volume>
+    <volume>0.000000001</volume>
+</link>
+<link name="camera_fwd_port_link">
+    <center_of_volume>0 0 0</center_of_volume>
+    <volume>0.000000001</volume>
+</link>
+<link name="camera_fwd_stbd_link">
+    <center_of_volume>0 0 0</center_of_volume>
+    <volume>0.000000001</volume>
+</link>
+<link name="camera_down_port_link">
+    <center_of_volume>0 0 0</center_of_volume>
+    <volume>0.000000001</volume>
+</link>
+<link name="camera_down_stbd_link">
+    <center_of_volume>0 0 0</center_of_volume>
+    <volume>0.000000001</volume>
+</link> -->
 </plugin>
 </gazebo>
-<!--                                -->
-<!-- Gazebo Riptide Link Properties -->
-<!--                                -->
-<gazebo reference="housing_link">
-  <material>Gazebo/Grey</material>
-</gazebo>
-<gazebo reference="chassis_link">
-  <material>Gazebo/FlatBlack</material>
-</gazebo>
-<gazebo reference="acoustics_link">
-  <material>Gazebo/DarkGrey</material>
-</gazebo>
-<gazebo reference="pneumatics_link">
-  <material>Gazebo/DarkGrey</material>
-</gazebo>
-<gazebo reference="port_battery_link">
-  <material>Gazebo/DarkGrey</material>
-</gazebo>
-<gazebo reference="stbd_battery_link">
-  <material>Gazebo/DarkGrey</material>
-</gazebo>
-<xacro:macro name="thruster_link_gazebo" params="name">
-  <gazebo reference="${name}_link">
-    <material>Gazebo/RedBright</material>
-  </gazebo>
-</xacro:macro>
-<xacro:thruster_link_gazebo name="surge_port_hi" />
-<xacro:thruster_link_gazebo name="surge_stbd_hi" />
-<xacro:thruster_link_gazebo name="surge_port_lo" />
-<xacro:thruster_link_gazebo name="surge_stbd_lo" />
-<xacro:thruster_link_gazebo name="sway_fwd" />
-<xacro:thruster_link_gazebo name="sway_aft" />
-<xacro:thruster_link_gazebo name="heave_port_fwd" />
-<xacro:thruster_link_gazebo name="heave_stbd_fwd" />
-<xacro:thruster_link_gazebo name="heave_port_aft" />
-<xacro:thruster_link_gazebo name="heave_stbd_aft" />
-<!--                                 -->
-<!-- Gazebo Riptide Joint Properties -->
-<!--                                 -->
-<gazebo reference="housing_imu_one_joint">
-  <disableFixedJointLumping>true</disableFixedJointLumping>
-</gazebo>
-<gazebo reference="housing_camera_fwd_port_joint">
-  <disableFixedJointLumping>true</disableFixedJointLumping>
-</gazebo>
-<gazebo reference="housing_camera_fwd_stbd_joint">
-  <disableFixedJointLumping>true</disableFixedJointLumping>
-</gazebo>
-<gazebo reference="housing_camera_down_port_joint">
-  <disableFixedJointLumping>true</disableFixedJointLumping>
-</gazebo>
-<gazebo reference="housing_camera_down_stbd_joint">
-  <disableFixedJointLumping>true</disableFixedJointLumping>
-</gazebo>
-<gazebo reference="base_housing_joint">
-  <disableFixedJointLumping>true</disableFixedJointLumping>
-</gazebo>
-<gazebo reference="housing_chassis_joint">
-  <disableFixedJointLumping>true</disableFixedJointLumping>
-</gazebo>
-<gazebo reference="chassis_acoustics_joint">
-  <disableFixedJointLumping>true</disableFixedJointLumping>
-</gazebo>
-<gazebo reference="chassis_pneumatics_joint">
-  <disableFixedJointLumping>true</disableFixedJointLumping>
-</gazebo>
-<gazebo reference="chassis_port_battery_joint">
-  <disableFixedJointLumping>true</disableFixedJointLumping>
-</gazebo>
-<gazebo reference="chassis_stbd_battery_joint">
-  <disableFixedJointLumping>true</disableFixedJointLumping>
-</gazebo>
-<xacro:macro name="thruster_joint_gazebo" params="name">
-  <gazebo reference="${name}_joint">
-    <disableFixedJointLumping>true</disableFixedJointLumping>
-  </gazebo>
-</xacro:macro>
-<xacro:thruster_joint_gazebo name="surge_port_hi" />
-<xacro:thruster_joint_gazebo name="surge_stbd_hi" />
-<xacro:thruster_joint_gazebo name="surge_port_lo" />
-<xacro:thruster_joint_gazebo name="surge_stbd_lo" />
-<xacro:thruster_joint_gazebo name="sway_fwd" />
-<xacro:thruster_joint_gazebo name="sway_aft" />
-<xacro:thruster_joint_gazebo name="heave_port_fwd" />
-<xacro:thruster_joint_gazebo name="heave_stbd_fwd" />
-<xacro:thruster_joint_gazebo name="heave_port_aft" />
-<xacro:thruster_joint_gazebo name="heave_stbd_aft" />
 <!--                                  -->
 <!-- Gazebo Riptide Camera Properties -->
