Commit message: Fixed URDF, messed up in previous commit

File: riptide_description/urdf/riptide_properties.xacro (robot description, xacro)
@@ -1,78 +1,80 @@
 <?xml version="1.0"?>
 <robot xmlns:xacro="http://ros.org/wiki/xacro">
-  <xacro:property name="housing_camera_fwd_port" value="0.8600 -0.2500 0.4100" />
-<xacro:property name="housing_camera_fwd_stbd" value="0.8600 0.1500 0.4100" />
-<xacro:property name="housing_camera_down_port" value="0.7700 0.2000 0.3300" />
-<xacro:property name="housing_camera_down_stbd" value="0.7700 0.2000 0.3300" />
-<xacro:property name="housing_depth_sensor" value="0.5900 0.1900 0.2700" />
-<xacro:property name="housing_imu_one" value="0.8000 0.2500 0.3500" />
-<xacro:property name="housing_imu_two" value="0.0000 0.0000 0.0000" />
-<xacro:property name="base_housing" value="-0.5400 -0.2000 -0.3500" />
-<xacro:property name="housing_chassis" value="0.9400 -0.5200 -0.0700" />
-<xacro:property name="chassis_acoustics" value="-0.3300 0.4600 0.3700" />
-<xacro:property name="chassis_pneumatics" value="-0.6600 0.7000 0.4000" />
-<xacro:property name="chassis_port_battery" value="-0.7100 0.6100 0.4400" />
-<xacro:property name="chassis_stbd_battery" value="-0.2600 0.5200 0.5000" />
-<xacro:property name="chassis_surge_port_hi" value="0.0000 0.0000 0.0000" />
-<xacro:property name="chassis_surge_stbd_hi" value="0.0000 0.0000 0.0000" />
-<xacro:property name="chassis_surge_port_lo" value="-0.5900 0.9100 0.2800" />
-<xacro:property name="chassis_surge_stbd_lo" value="-0.5900 0.5300 0.2800" />
-<xacro:property name="chassis_sway_fwd" value="-0.3000 0.5800 0.2900" />
-<xacro:property name="chassis_sway_aft" value="-0.7700 0.5800 0.2900" />
-<xacro:property name="chassis_heave_port_fwd" value="-0.1300 0.9100 0.4200" />
-<xacro:property name="chassis_heave_stbd_fwd" value="-0.1300 0.5300 0.4200" />
-<xacro:property name="chassis_heave_port_aft" value="-0.6700 0.9100 0.4200" />
-<xacro:property name="chassis_heave_stbd_aft" value="-0.6700 0.5300 0.4200" />
-<xacro:property name="housing_com" value="0.1900 0.4100 0.5600" />
-<xacro:property name="chassis_com" value="0.4000 0.3500 0.5800" />
-<xacro:property name="acoustics_com" value="0.0600 0.0700 0.1200" />
-<xacro:property name="pneumatics_com" value="0.1200 0.1000 0.1500" />
-<xacro:property name="port_battery_com" value="0.0600 0.1500 0.2100" />
-<xacro:property name="stbd_battery_com" value="0.1100 0.1300 0.2400" />
-<xacro:property name="thruster_com" value="0.0000 0.0006 0.0075" />
-<xacro:property name="housing_mass" value="15.9700" />
-<xacro:property name="chassis_mass" value="3.9300" />
-<xacro:property name="acoustics_mass" value="0.9700" />
-<xacro:property name="pneumatics_mass" value="1.3500" />
-<xacro:property name="port_battery_mass" value="1.8700" />
-<xacro:property name="stbd_battery_mass" value="1.8600" />
-<xacro:property name="thruster_mass" value="0.3518" />
-<xacro:property name="housing_inertia"><inertia ixx="8.2500" ixy="0.0000" ixz="0.0000" iyy="6.2300" iyz="0.0000" izz="3.4600" /></xacro:property>
-<xacro:property name="chassis_inertia"><inertia ixx="1.8800" ixy="0.0000" ixz="0.0000" iyy="2.2000" iyz="0.0000" izz="1.3500" /></xacro:property>
-<xacro:property name="acoustics_inertia"><inertia ixx="0.0200" ixy="0.0000" ixz="0.0000" iyy="0.0200" iyz="0.0000" izz="0.0100" /></xacro:property>
-<xacro:property name="pneumatics_inertia"><inertia ixx="0.0500" ixy="0.0000" ixz="0.0000" iyy="0.0600" iyz="0.0000" izz="0.0400" /></xacro:property>
-<xacro:property name="port_battery_inertia"><inertia ixx="0.1300" ixy="0.0000" ixz="0.0000" iyy="0.1000" iyz="0.0000" izz="0.0500" /></xacro:property>
-<xacro:property name="stbd_battery_inertia"><inertia ixx="0.1500" ixy="0.0000" ixz="0.0000" iyy="0.1400" iyz="0.0000" izz="0.0600" /></xacro:property>
-<xacro:property name="thruster_inertia"><inertia ixx="0.0003" ixy="0.0000" ixz="0.0000" iyy="0.0003" iyz="0.0000" izz="0.0003" /></xacro:property>
-<xacro:property name="housing_cov" value="0.0000 0.0000 0.0000" />
-<xacro:property name="chassis_cov" value="0.0000 0.0000 0.0000" />
-<xacro:property name="acoustics_cov" value="0.0000 0.0000 0.0000" />
-<xacro:property name="pneumatics_cov" value="0.0000 0.0000 0.0000" />
-<xacro:property name="port_battery_cov" value="0.0000 0.0000 0.0000" />
-<xacro:property name="stbd_battery_cov" value="0.0000 0.0000 0.0000" />
-<xacro:property name="thruster_cov" value="0.0000 0.0006 0.0075" />
-<xacro:property name="housing_volume" value="0.0000" />
-<xacro:property name="chassis_volume" value="0.0000" />
-<xacro:property name="acoustics_volume" value="0.0000" />
-<xacro:property name="pneumatics_volume" value="0.0000" />
-<xacro:property name="port_battery_volume" value="0.0000" />
-<xacro:property name="stbd_battery_volume" value="0.0000" />
-<xacro:property name="thruster_volume" value="0.0002" />
-<xacro:property name="housing_mesh" value="package://riptide_description/meshes/housing.stl" />
-<xacro:property name="chassis_mesh" value="package://riptide_description/meshes/chassis.stl" />
-<xacro:property name="acoustics_mesh" value="package://riptide_description/meshes/acoustics.stl" />
-<xacro:property name="pneumatics_mesh" value="package://riptide_description/meshes/pneumatics.stl" />
-<xacro:property name="port_battery_mesh" value="package://riptide_description/meshes/port_battery.stl" />
-<xacro:property name="stbd_battery_mesh" value="package://riptide_description/meshes/stbd_battery.stl" />
-<xacro:property name="thruster_mesh" value="package://riptide_description/meshes/thruster.stl" />
-<xacro:property name="align_surge_port_hi" value="0 ${-M_PI/2} ${M_PI}" />
-<xacro:property name="align_surge_stbd_hi" value="0 ${M_PI/2} 0" />
-<xacro:property name="align_surge_port_lo" value="0 ${-M_PI/2} ${M_PI}" />
-<xacro:property name="align_surge_stbd_lo" value="0 ${M_PI/2} 0" />
-<xacro:property name="align_sway_fwd" value="0 ${M_PI/2} ${M_PI/2}" />
-<xacro:property name="align_sway_aft" value="0 ${-M_PI/2} ${-M_PI/2}" />
-<xacro:property name="align_heave_port_fwd" value="0 0 ${M_PI}" />
-<xacro:property name="align_heave_stbd_fwd" value="0 0 0" />
-<xacro:property name="align_heave_port_aft" value="0 0 ${M_PI}" />
-<xacro:property name="align_heave_stbd_aft" value="0 0 0" />
+  <xacro:property name="housing_camera_fwd_port" value="0.4 0.0400 -0.0004" />
+  <xacro:property name="housing_camera_fwd_stbd" value="0.4 -0.0400 -0.0004" />
+  <xacro:property name="housing_camera_down_port" value="0.2360 0.0400 -0.0620" />
+  <xacro:property name="housing_camera_down_stbd" value="0.2360 -0.0400 -0.0620" />
+  <xacro:property name="housing_depth_sensor" value="0.0000 0.0000 0.1049" />
+  <xacro:property name="housing_imu_one" value="0.1322 -0.0056 0.0268" />
+  <xacro:property name="housing_imu_two" value="-0.1469 0.0004 -0.0405" />
+  <xacro:property name="housing_camera_left" value="0 0 -0.2" />
+  <xacro:property name="housing_camera_right" value="0 0 0.2" />
+  <xacro:property name="base_housing" value="0.0737 0.0005 0.0621" />
+  <xacro:property name="housing_chassis" value="-0.0556 0.0000 -0.0749" />
+  <xacro:property name="chassis_acoustics" value="0.1699 0.0000 -0.0584" />
+  <xacro:property name="chassis_pneumatics" value="-0.1172 0.0000 -0.0584" />
+  <xacro:property name="chassis_port_battery" value="-0.1781 0.1302 -0.0140" />
+  <xacro:property name="chassis_stbd_battery" value="-0.1781 -0.1302 -0.0140" />
+  <xacro:property name="chassis_surge_port_hi" value="-0.2238 0.1824 0.1384" />
+  <xacro:property name="chassis_surge_stbd_hi" value="-0.2238 -0.1824 0.1384" />
+  <xacro:property name="chassis_surge_port_lo" value="-0.2238 0.1824 -0.0838" />
+  <xacro:property name="chassis_surge_stbd_lo" value="-0.2238 -0.1824 -0.0838" />
+  <xacro:property name="chassis_sway_fwd" value="0.3776 0.0000 -0.0838" />
+  <xacro:property name="chassis_sway_aft" value="-0.3744 0.0000 -0.0838" />
+  <xacro:property name="chassis_heave_port_fwd" value="0.2824 0.1824 -0.0033" />
+  <xacro:property name="chassis_heave_stbd_fwd" value="0.2824 -0.1824 -0.0033" />
+  <xacro:property name="chassis_heave_port_aft" value="-0.2724 0.1824 -0.0033" />
+  <xacro:property name="chassis_heave_stbd_aft" value="-0.2724 -0.1824 -0.0033" />
+  <xacro:property name="housing_com" value="-0.0434 0.0009 -0.0155" />
+  <xacro:property name="chassis_com" value="-0.0129 0.0000 -0.0561" />
+  <xacro:property name="acoustics_com" value="0.0027 0.0027 -0.0265" />
+  <xacro:property name="pneumatics_com" value="0.0141 0.0015 -0.0392" />
+  <xacro:property name="port_battery_com" value="0.0936 0.0278 -0.0003" />
+  <xacro:property name="stbd_battery_com" value="0.0936 -0.0278 -0.0003" />
+  <xacro:property name="thruster_com" value="0.0000 0.0006 0.0075" />
+  <xacro:property name="housing_mass" value="14.3153" />
+  <xacro:property name="chassis_mass" value="2.7134" />
+  <xacro:property name="acoustics_mass" value="0.9657" />
+  <xacro:property name="pneumatics_mass" value="1.3503" />
+  <xacro:property name="port_battery_mass" value="1.8671" />
+  <xacro:property name="stbd_battery_mass" value="1.8671" />
+  <xacro:property name="thruster_mass" value="0.3518" />
+  <xacro:property name="housing_inertia"><inertia ixx="0.1230" ixy="0.0000" ixz="0.0000" iyy="0.6568" iyz="0.0000" izz="0.6422" /></xacro:property>
+  <xacro:property name="chassis_inertia"><inertia ixx="0.0572" ixy="0.0000" ixz="0.0000" iyy="0.1657" iyz="0.0000" izz="0.1830" /></xacro:property>
+  <xacro:property name="acoustics_inertia"><inertia ixx="0.0026" ixy="0.0000" ixz="0.0000" iyy="0.0026" iyz="0.0000" izz="0.0030" /></xacro:property>
+  <xacro:property name="pneumatics_inertia"><inertia ixx="0.0080" ixy="0.0000" ixz="0.0000" iyy="0.0088" iyz="0.0000" izz="0.0107" /></xacro:property>
+  <xacro:property name="port_battery_inertia"><inertia ixx="0.0034" ixy="0.0000" ixz="0.0000" iyy="0.0253" iyz="0.0000" izz="0.0262" /></xacro:property>
+  <xacro:property name="stbd_battery_inertia"><inertia ixx="0.0034" ixy="0.0000" ixz="0.0000" iyy="0.0253" iyz="0.0000" izz="0.0262" /></xacro:property>
+  <xacro:property name="thruster_inertia"><inertia ixx="0.0003" ixy="0.0000" ixz="0.0000" iyy="0.0003" iyz="0.0000" izz="0.0003" /></xacro:property>
+  <xacro:property name="housing_cov" value="-0.0480 0.0000 -0.0037" />
+  <xacro:property name="chassis_cov" value="-0.0120 0.0000 -0.0566" />
+  <xacro:property name="acoustics_cov" value="0.0014 0.0014 -0.0277" />
+  <xacro:property name="pneumatics_cov" value="0.0025 0.0002 -0.0369" />
+  <xacro:property name="port_battery_cov" value="0.1257 0.0335 -0.0001" />
+  <xacro:property name="stbd_battery_cov" value="0.1257 -0.0335 -0.0001" />
+  <xacro:property name="thruster_cov" value="0.0000 0.0006 0.0075" />
+  <xacro:property name="housing_volume" value="0.0262" />
+  <xacro:property name="chassis_volume" value="0.0010" />
+  <xacro:property name="acoustics_volume" value="0.0010" />
+  <xacro:property name="pneumatics_volume" value="0.0024" />
+  <xacro:property name="port_battery_volume" value="0.0013" />
+  <xacro:property name="stbd_battery_volume" value="0.0013" />
+  <xacro:property name="thruster_volume" value="0.0002" />
+  <xacro:property name="housing_mesh" value="package://riptide_description/meshes/housing.stl" />
+  <xacro:property name="chassis_mesh" value="package://riptide_description/meshes/chassis.stl" />
+  <xacro:property name="acoustics_mesh" value="package://riptide_description/meshes/acoustics.stl" />
+  <xacro:property name="pneumatics_mesh" value="package://riptide_description/meshes/pneumatics.stl" />
+  <xacro:property name="port_battery_mesh" value="package://riptide_description/meshes/port_battery.stl" />
+  <xacro:property name="stbd_battery_mesh" value="package://riptide_description/meshes/stbd_battery.stl" />
+  <xacro:property name="thruster_mesh" value="package://riptide_description/meshes/thruster.stl" />
+  <xacro:property name="align_surge_port_hi" value="0 ${-M_PI/2} ${M_PI}" />
+  <xacro:property name="align_surge_stbd_hi" value="0 ${M_PI/2} 0" />
+  <xacro:property name="align_surge_port_lo" value="0 ${-M_PI/2} ${M_PI}" />
+  <xacro:property name="align_surge_stbd_lo" value="0 ${M_PI/2} 0" />
+  <xacro:property name="align_sway_fwd" value="0 ${M_PI/2} ${M_PI/2}" />
+  <xacro:property name="align_sway_aft" value="0 ${-M_PI/2} ${-M_PI/2}" />
+  <xacro:property name="align_heave_port_fwd" value="0 0 ${M_PI}" />
+  <xacro:property name="align_heave_stbd_fwd" value="0 0 0" />
+  <xacro:property name="align_heave_port_aft" value="0 0 ${M_PI}" />
+  <xacro:property name="align_heave_stbd_aft" value="0 0 0" />
 </robot>
