Commit message: Hotfix: URDF error leftover from merge

File: riptide_description/urdf/riptide_links.xacro (robot description, xacro)
@@ -5,16 +5,4 @@
   <!--                             -->
   <link name="base_link">
-    <inertial>
-      <mass value="0.00001" />
-      <inertia ixx="0.0" ixy="0.0" ixz="0.0" iyy="0.0" iyz="0.0" izz="0.0" />
-    </inertial>
-  </link>
-  <link name="camera_left">
-    <inertial>
-      <mass value="0.00001" />
-      <inertia ixx="0.0" ixy="0.0" ixz="0.0" iyy="0.0" iyz="0.0" izz="0.0" />
-    </inertial>
-  </link>
-  <link name="camera_right">
     <inertial>
       <mass value="0.00001" />

Commit message: Fixing simulator

File: riptide_description/urdf/riptide_links.xacro (robot description, xacro)
@@ -9,4 +9,10 @@
       <inertia ixx="0.0" ixy="0.0" ixz="0.0" iyy="0.0" iyz="0.0" izz="0.0" />
     </inertial>
+    <!-- <buoyancy>
+    <compensation>10000</compensation>
+      <origin xyz= "0 0 0"/>
+      <limit radius=".25"/>
+      <damping xyz="60 100 100" rpy="20 50 50"/>
+    </buoyancy> -->
   </link>
   <!--               -->

File: riptide_description/urdf/riptide_simulation.xacro (robot description, xacro)
@@ -129,5 +129,5 @@
     <!-- Gazebo Riptide Buoyancy Properties -->
     <!--                                    -->
-    <plugin name="BuoyancyPlugin" filename="libBuoyancyPlugin.so">
+    <!--<plugin name="BuoyancyPlugin" filename="libBuoyancyPlugin.so">
       <robotNamespace></robotNamespace>
       <fluid_density>108</fluid_density>
@@ -200,5 +200,5 @@
         <volume>0.000000001</volume>
       </link>
-    </plugin>
+    </plugin>-->
   </gazebo>
   <!--                                  -->

Commit message: Added buoyancy plugin!

File: riptide_description/urdf/riptide_links.xacro (robot description, xacro)
@@ -9,10 +9,4 @@
       <inertia ixx="0.0" ixy="0.0" ixz="0.0" iyy="0.0" iyz="0.0" izz="0.0" />
     </inertial>
-    <!-- <buoyancy>
-    <compensation>10000</compensation>
-      <origin xyz= "0 0 0"/>
-      <limit radius=".25"/>
-      <damping xyz="60 100 100" rpy="20 50 50"/>
-    </buoyancy> -->
   </link>
   <!--               -->
@@ -36,4 +30,10 @@
       </geometry>
     </collision>
+    <buoyancy>
+      <compensation>2</compensation>
+      <origin xyz= "${housing_com}"/>
+      <limit radius=".25"/>
+      <damping xyz="60 100 100" rpy="20 50 50"/>
+    </buoyancy>
   </link>
   <link name="chassis_link">
@@ -72,4 +72,10 @@
       </geometry>
     </collision>
+    <buoyancy>
+      <compensation>0</compensation>
+      <origin xyz= "${acoustics_com}"/>
+      <limit radius=".25"/>
+      <damping xyz="60 100 100" rpy="20 50 50"/>
+    </buoyancy>
   </link>
   <link name="pneumatics_link">
@@ -90,4 +96,10 @@
       </geometry>
     </collision>
+    <buoyancy>
+      <compensation>2</compensation>
+      <origin xyz= "${pneumatics_com}"/>
+      <limit radius=".25"/>
+      <damping xyz="60 100 100" rpy="20 50 50"/>
+    </buoyancy>
   </link>
   <link name="port_battery_link">
@@ -108,4 +120,10 @@
       </geometry>
     </collision>
+    <buoyancy>
+      <compensation>1.5</compensation>
+      <origin xyz= "${port_battery_com}"/>
+      <limit radius=".25"/>
+      <damping xyz="60 100 100" rpy="20 50 50"/>
+    </buoyancy>
   </link>
   <link name="stbd_battery_link">
@@ -126,5 +144,11 @@
       </geometry>
     </collision>
-  </link> -->
+    <buoyancy>
+      <compensation>1.5</compensation>
+      <origin xyz= "${stbd_battery_com}"/>
+      <limit radius=".25"/>
+      <damping xyz="60 100 100" rpy="20 50 50"/>
+    </buoyancy>
+  </link>
   <!--                -->
   <!-- Thruster Links -->
