Commit message: Added functional IMU.

File: riptide_description/urdf/riptide_joints.xacro (robot description, xacro)
@@ -8,4 +8,12 @@
     <parent link="base_link"/>
     <child link="housing_link"/>
+  </joint>
+  <!--               -->
+  <!-- Sensor Joints -->
+  <!--               -->
+  <joint name="housing_imu_one_joint" type="fixed">
+    <origin xyz="${housing_imu_one}" rpy="0 0 0" />
+    <parent link="housing_link"/>
+    <child link="imu_one_link"/>
   </joint>
   <!--                -->

File: riptide_description/urdf/riptide_links.xacro (robot description, xacro)
@@ -7,4 +7,13 @@
     <inertial>
       <mass value="8.3901" />
+      <inertia ixx="0.0" ixy="0.0" ixz="0.0" iyy="0.0" iyz="0.0" izz="0.0" />
+    </inertial>
+  </link>
+  <!--              -->
+  <!-- Sensor Links -->
+  <!--              -->
+  <link name="imu_one_link">
+    <inertial>
+      <mass value="0.00001" />
       <inertia ixx="0.0" ixy="0.0" ixz="0.0" iyy="0.0" iyz="0.0" izz="0.0" />
     </inertial>

File: riptide_description/urdf/riptide_simulation.xacro (robot description, xacro)
@@ -5,8 +5,26 @@
     <!--                                 -->
   <gazebo>
+    <!--                                  -->
+    <!-- Gazebo Riptide Sensor Properties -->
+    <!--                                  -->
+    <plugin name="imu_one" filename="libgazebo_ros_imu.so">
+      <robotNamespace></robotNamespace>
+      <serviceName>/imu</serviceName>
+      <topicName>/state/imu</topicName>
+      <gaussianNoise>0.0</gaussianNoise>
+      <bodyName>imu_one_link</bodyName>
+      <xyzOffset>0 0 0</xyzOffset>
+      <rpyOffset>0 0 0</rpyOffset>
+      <updateRate>100.0</updateRate>
+      <frameName>imu_one_link</frameName>
+    </plugin>
     <!--                                    -->
     <!-- Gazebo Riptide Buoyancy Properties -->
     <!--                                    -->
     <plugin name="BuoyancyPlugin" filename="libBuoyancyPlugin.so">
+      <link name="imu_one_link">
+        <center_of_volume>0 0 0</center_of_volume>
+        <volume>0.0000000001</volume>
+      </link>
       <link name="base_link">
         <center_of_volume>0 0 0</center_of_volume>
@@ -94,4 +112,7 @@
     <!-- Gazebo Riptide Joint Properties -->
     <!--                                 -->
+    <gazebo reference="housing_imu_one_joint">
+      <disableFixedJointLumping>true</disableFixedJointLumping>
+    </gazebo>
     <gazebo reference="base_housing_joint">
       <disableFixedJointLumping>true</disableFixedJointLumping>

Commit message: Added experimental state machine command server

File: riptide_description/urdf/riptide_joints.xacro (robot description, xacro)
@@ -16,4 +16,14 @@
     <parent link="housing_link"/>
     <child link="imu_one_link"/>
+  </joint>
+  <joint name="housing_camera_left_joint" type="fixed">
+    <origin xyz="${housing_camera_left}" rpy="0 0 0" />
+    <parent link="housing_link"/>
+    <child link="camera_left"/>
+  </joint>
+  <joint name="housing_camera_right_joint" type="fixed">
+    <origin xyz="${housing_camera_right}" rpy="0 0 0" />
+    <parent link="housing_link"/>
+    <child link="camera_right"/>
   </joint>
   <!--                -->

File: riptide_description/urdf/riptide_links.xacro (robot description, xacro)
@@ -14,4 +14,16 @@
   <!--              -->
   <link name="imu_one_link">
+    <inertial>
+      <mass value="0.00001" />
+      <inertia ixx="0.0" ixy="0.0" ixz="0.0" iyy="0.0" iyz="0.0" izz="0.0" />
+    </inertial>
+  </link>
+  <link name="camera_left">
+    <inertial>
+      <mass value="0.00001" />
+      <inertia ixx="0.0" ixy="0.0" ixz="0.0" iyy="0.0" iyz="0.0" izz="0.0" />
+    </inertial>
+  </link>
+  <link name="camera_right">
     <inertial>
       <mass value="0.00001" />

File: riptide_description/urdf/riptide_properties.xacro (robot description, xacro)
@@ -7,4 +7,6 @@
   <xacro:property name="housing_imu_one" value="0.1322 -0.0056 0.0268" />
   <xacro:property name="housing_imu_two" value="-0.1469 0.0004 -0.0405" />
+  <xacro:property name="housing_camera_left" value="0 0 -0.2" />
+  <xacro:property name="housing_camera_right" value="0 0 0.2" />
   <xacro:property name="base_housing" value="0.0737 0.0005 0.0621" />
   <xacro:property name="housing_chassis" value="-0.0556 0.0000 -0.0749" />

Commit message: Added depth sensor plugin. Removed buoyancy and gravity for testing.

File: riptide_description/urdf/riptide_joints.xacro (robot description, xacro)
@@ -65,4 +65,9 @@
       <child link="imu_one_link"/>
     </joint>
+    <joint name="housing_depth_sensor_joint" type="fixed">
+      <origin xyz="${housing_depth_sensor}" rpy="0 0 0" />
+      <parent link="housing_link"/>
+      <child link="depth_sensor_link"/>
+    </joint>
     <joint name="housing_camera_fwd_port_joint" type="fixed">
       <origin xyz="${housing_camera_fwd_port}" rpy="0 0 0" />

File: riptide_description/urdf/riptide_links.xacro (robot description, xacro)
@@ -159,5 +159,17 @@
   <link name="imu_one_link">
     <inertial>
-      <mass value="8" />
+      <mass value="0.00001" />
+      <inertia ixx="0.0" ixy="0.0" ixz="0.0" iyy="0.0" iyz="0.0" izz="0.0" />
+    </inertial>
+    <!-- Collision Geometry necessary for Buoyancy Plugin to work! -->
+    <collision>
+      <geometry>
+        <box size="0.0001 0.0001 0.0001" />
+      </geometry>
+    </collision>
+  </link>
+  <link name="depth_sensor_link">
+    <inertial>
+      <mass value="0.00001" />
       <inertia ixx="0.0" ixy="0.0" ixz="0.0" iyy="0.0" iyz="0.0" izz="0.0" />
     </inertial>

File: riptide_description/urdf/riptide_simulation.xacro (robot description, xacro)
@@ -73,19 +73,22 @@
   <xacro:thruster_joint_gazebo name="heave_port_aft" />
   <xacro:thruster_joint_gazebo name="heave_stbd_aft" /> -->
-    <gazebo reference="housing_imu_one_joint">
-      <disableFixedJointLumping>true</disableFixedJointLumping>
-    </gazebo>
-    <gazebo reference="housing_camera_fwd_port_joint">
-      <disableFixedJointLumping>true</disableFixedJointLumping>
-    </gazebo>
-    <gazebo reference="housing_camera_fwd_stbd_joint">
-      <disableFixedJointLumping>true</disableFixedJointLumping>
-    </gazebo>
-    <gazebo reference="housing_camera_down_port_joint">
-      <disableFixedJointLumping>true</disableFixedJointLumping>
-    </gazebo>
-    <gazebo reference="housing_camera_down_stbd_joint">
-      <disableFixedJointLumping>true</disableFixedJointLumping>
-    </gazebo>
+  <gazebo reference="housing_imu_one_joint">
+    <disableFixedJointLumping>true</disableFixedJointLumping>
+  </gazebo>
+  <gazebo reference="housing_depth_sensor_joint">
+    <disableFixedJointLumping>true</disableFixedJointLumping>
+  </gazebo>
+  <gazebo reference="housing_camera_fwd_port_joint">
+    <disableFixedJointLumping>true</disableFixedJointLumping>
+  </gazebo>
+  <gazebo reference="housing_camera_fwd_stbd_joint">
+    <disableFixedJointLumping>true</disableFixedJointLumping>
+  </gazebo>
+  <gazebo reference="housing_camera_down_port_joint">
+    <disableFixedJointLumping>true</disableFixedJointLumping>
+  </gazebo>
+  <gazebo reference="housing_camera_down_stbd_joint">
+    <disableFixedJointLumping>true</disableFixedJointLumping>
+  </gazebo>
   <!--                                 -->
   <!--  Riptide Simulation Properties  -->
@@ -95,5 +98,4 @@
     <!-- Gazebo Riptide Sensor Properties -->
     <!--                                  -->
-<!--
     <plugin name="imu_one" filename="libgazebo_ros_imu.so">
       <robotNamespace></robotNamespace>
@@ -106,142 +108,155 @@
       <updateRate>100.0</updateRate>
       <frameName>imu_one_link</frameName>
-    </plugin> -->
+    </plugin>
     <!--                                    -->
     <!-- Gazebo Riptide Thruster Properties -->
     <!--                                    -->
-<!--
     <plugin filename="libgazebo_ros_riptide_thrust.so" name="thrust">
       <robotNamespace></robotNamespace>
       <topicName>/command/thrust</topicName>
-    </plugin> -->
+    </plugin>
+    <!--                                    -->
+    <!-- Gazebo Riptide Depth Sensor Properties -->
+    <!--                                    -->
+    <plugin filename="libgazebo_ros_depth_sensor.so" name="DepthSensor">
+      <robotNamespace></robotNamespace>
+      <topicName>/state/depth</topicName>
+      <seaLevel>20</seaLevel>
+      <fluidDensity>1</fluidDensity>
+      <sensorLink>depth_sensor_link</sensorLink>
+    </plugin>
     <!--                                    -->
     <!-- Gazebo Riptide Buoyancy Properties -->
     <!--                                    -->
-<plugin name="BuoyancyPlugin" filename="libBuoyancyPlugin.so">
-<robotNamespace></robotNamespace>
-<fluid_density>195</fluid_density>
-<link name="base_link">
-  <center_of_volume>0 0 0</center_of_volume>
-  <volume>0.000000001</volume>
-</link>
-<link name="housing_link">
-<center_of_volume>${housing_cov}</center_of_volume>
-<volume>${housing_volume}</volume>
-</link>
-<link name="chassis_link">
-<center_of_volume>${chassis_cov}</center_of_volume>
-<volume>${chassis_volume}</volume>
-</link>
-<link name="acoustics_link">
-<center_of_volume>${acoustics_cov}</center_of_volume>
-<volume>${acoustics_volume}</volume>
-</link>
-<link name="pneumatics_link">
-<center_of_volume>${pneumatics_cov}</center_of_volume>
-<volume>${pneumatics_volume}</volume>
-</link>
-<link name="port_battery_link">
-<center_of_volume>${port_battery_cov}</center_of_volume>
-<volume>${port_battery_volume}</volume>
-</link>
-<link name="stbd_battery_link">
-<center_of_volume>${stbd_battery_cov}</center_of_volume>
-<volume>${stbd_battery_volume}</volume>
-</link>
-<xacro:macro name="thruster_volume" params="thruster">
-<link name="${thruster}_link">
-<center_of_volume>${thruster_cov}</center_of_volume>
-<volume>${thruster_volume}</volume>
-</link>
-</xacro:macro>
-<xacro:thruster_volume thruster="surge_port_hi" />
-<xacro:thruster_volume thruster="surge_stbd_hi" />
-<xacro:thruster_volume thruster="surge_port_lo" />
-<xacro:thruster_volume thruster="surge_stbd_lo" />
-<xacro:thruster_volume thruster="sway_fwd" />
-<xacro:thruster_volume thruster="sway_aft" />
-<xacro:thruster_volume thruster="heave_port_fwd" />
-<xacro:thruster_volume thruster="heave_stbd_fwd" />
-<xacro:thruster_volume thruster="heave_port_aft" />
-<xacro:thruster_volume thruster="heave_stbd_aft" />
-<link name="imu_one_link">
-    <center_of_volume>0 0 0</center_of_volume>
-    <volume>0.000000001</volume>
-</link>
-<link name="camera_fwd_port_link">
-    <center_of_volume>0 0 0</center_of_volume>
-    <volume>0.000000001</volume>
-</link>
-<link name="camera_fwd_stbd_link">
-    <center_of_volume>0 0 0</center_of_volume>
-    <volume>0.000000001</volume>
-</link>
-<link name="camera_down_port_link">
-    <center_of_volume>0 0 0</center_of_volume>
-    <volume>0.000000001</volume>
-</link>
-<link name="camera_down_stbd_link">
-    <center_of_volume>0 0 0</center_of_volume>
-    <volume>0.000000001</volume>
-</link> -->
-</plugin>
-</gazebo>
-<!--                                  -->
-<!-- Gazebo Riptide Camera Properties -->
-<!--                                  -->
-<!-- Camera 1 -->
-<gazebo reference="camera_fwd_port_link">
-  <sensor type="multicamera" name="stereo_camera">
-    <update_rate>30.0</update_rate>
-    <camera name="left">
-      <horizontal_fov>1.3962634</horizontal_fov>
-      <image>
-        <width>800</width>
-        <height>800</height>
-        <format>R8G8B8</format>
-      </image>
-      <clip>
-        <near>0.02</near>
-        <far>300</far>
-      </clip>
-      <noise>
-        <type>gaussian</type>
-        <mean>0.0</mean>
-        <stddev>0.007</stddev>
-      </noise>
-    </camera>
-    <camera name="right">
-      <pose>0 -0.07 0 0 0 0</pose>
-      <horizontal_fov>1.3962634</horizontal_fov>
-      <image>
-        <width>800</width>
-        <height>800</height>
-        <format>R8G8B8</format>
-      </image>
-      <clip>
-        <near>0.02</near>
-        <far>300</far>
-      </clip>
-      <noise>
-        <type>gaussian</type>
-        <mean>0.0</mean>
-        <stddev>0.007</stddev>
-      </noise>
-    </camera>
-    <plugin name="stereo_camera_controller" filename="libgazebo_ros_multicamera.so">
-      <alwaysOn>true</alwaysOn>
-      <updateRate>0.0</updateRate>
-      <cameraName>riptide/stereo_fwd</cameraName>
-      <imageTopicName>image_raw</imageTopicName>
-      <cameraInfoTopicName>camera_info</cameraInfoTopicName>
-      <frameName>camera_fwd_port_link</frameName>
-      <hackBaseline>0.07</hackBaseline>
-      <distortionK1>0.0</distortionK1>
-      <distortionK2>0.0</distortionK2>
-      <distortionK3>0.0</distortionK3>
-      <distortionT1>0.0</distortionT1>
-      <distortionT2>0.0</distortionT2>
-    </plugin>
-  </sensor>
-</gazebo>
+    <!--<plugin name="BuoyancyPlugin" filename="libBuoyancyPlugin.so">
+      <robotNamespace></robotNamespace>
+      <fluid_density>160</fluid_density>
+      <link name="base_link">
+        <center_of_volume>0 0 0</center_of_volume>
+        <volume>0.000000001</volume>
+      </link>
+      <link name="housing_link">
+        <center_of_volume>${housing_cov}</center_of_volume>
+        <volume>${housing_volume}</volume>
+      </link>
+      <link name="chassis_link">
+        <center_of_volume>${chassis_cov}</center_of_volume>
+        <volume>${chassis_volume}</volume>
+      </link>
+      <link name="acoustics_link">
+        <center_of_volume>${acoustics_cov}</center_of_volume>
+        <volume>${acoustics_volume}</volume>
+      </link>
+      <link name="pneumatics_link">
+        <center_of_volume>${pneumatics_cov}</center_of_volume>
+        <volume>${pneumatics_volume}</volume>
+      </link>
+      <link name="port_battery_link">
+        <center_of_volume>${port_battery_cov}</center_of_volume>
+        <volume>${port_battery_volume}</volume>
+      </link>
+      <link name="stbd_battery_link">
+        <center_of_volume>${stbd_battery_cov}</center_of_volume>
+        <volume>${stbd_battery_volume}</volume>
+      </link>
+      <xacro:macro name="thruster_volume" params="thruster">
+        <link name="${thruster}_link">
+          <center_of_volume>${thruster_cov}</center_of_volume>
+          <volume>${thruster_volume}</volume>
+        </link>
+      </xacro:macro>
+      <xacro:thruster_volume thruster="surge_port_hi" />
+      <xacro:thruster_volume thruster="surge_stbd_hi" />
+      <xacro:thruster_volume thruster="surge_port_lo" />
+      <xacro:thruster_volume thruster="surge_stbd_lo" />
+      <xacro:thruster_volume thruster="sway_fwd" />
+      <xacro:thruster_volume thruster="sway_aft" />
+      <xacro:thruster_volume thruster="heave_port_fwd" />
+      <xacro:thruster_volume thruster="heave_stbd_fwd" />
+      <xacro:thruster_volume thruster="heave_port_aft" />
+      <xacro:thruster_volume thruster="heave_stbd_aft" />
+      <link name="imu_one_link">
+        <center_of_volume>0 0 0</center_of_volume>
+        <volume>0.000000001</volume>
+      </link>
+      <link name="depth_sensor_link">
+        <center_of_volume>0 0 0</center_of_volume>
+        <volume>0.000000001</volume>
+      </link>
+      <link name="camera_fwd_port_link">
+        <center_of_volume>0 0 0</center_of_volume>
+        <volume>0.000000001</volume>
+      </link>
+      <link name="camera_fwd_stbd_link">
+        <center_of_volume>0 0 0</center_of_volume>
+        <volume>0.000000001</volume>
+      </link>
+      <link name="camera_down_port_link">
+        <center_of_volume>0 0 0</center_of_volume>
+        <volume>0.000000001</volume>
+      </link>
+      <link name="camera_down_stbd_link">
+        <center_of_volume>0 0 0</center_of_volume>
+        <volume>0.000000001</volume>
+      </link>
+    </plugin>-->
+  </gazebo>
+  <!--                                  -->
+  <!-- Gazebo Riptide Camera Properties -->
+  <!--                                  -->
+  <!-- Stereo Camera -->
+  <gazebo reference="camera_fwd_port_link">
+    <sensor type="multicamera" name="stereo_camera">
+      <update_rate>30.0</update_rate>
+      <camera name="left">
+        <horizontal_fov>1.3962634</horizontal_fov>
+        <image>
+          <width>800</width>
+          <height>800</height>
+          <format>R8G8B8</format>
+        </image>
+        <clip>
+          <near>0.02</near>
+          <far>300</far>
+        </clip>
+        <noise>
+          <type>gaussian</type>
+          <mean>0.0</mean>
+          <stddev>0.007</stddev>
+        </noise>
+      </camera>
+      <camera name="right">
+        <pose>0 -0.07 0 0 0 0</pose>
+        <horizontal_fov>1.3962634</horizontal_fov>
+        <image>
+          <width>800</width>
+          <height>800</height>
+          <format>R8G8B8</format>
+        </image>
+        <clip>
+          <near>0.02</near>
+          <far>300</far>
+        </clip>
+        <noise>
+          <type>gaussian</type>
+          <mean>0.0</mean>
+          <stddev>0.007</stddev>
+        </noise>
+      </camera>
+      <plugin name="stereo_camera_controller" filename="libgazebo_ros_multicamera.so">
+        <alwaysOn>true</alwaysOn>
+        <updateRate>0.0</updateRate>
+        <cameraName>riptide/stereo_fwd</cameraName>
+        <imageTopicName>image_raw</imageTopicName>
+        <cameraInfoTopicName>camera_info</cameraInfoTopicName>
+        <frameName>camera_fwd_port_link</frameName>
+        <hackBaseline>0.07</hackBaseline>
+        <distortionK1>0.0</distortionK1>
+        <distortionK2>0.0</distortionK2>
+        <distortionK3>0.0</distortionK3>
+        <distortionT1>0.0</distortionT1>
+        <distortionT2>0.0</distortionT2>
+      </plugin>
+    </sensor>
+  </gazebo>
 </robot>

Commit message: Removed surge highs

File: riptide_description/urdf/riptide_joints.xacro (robot description, xacro)
@@ -47,6 +47,4 @@
     </joint>
   </xacro:macro>
-  <xacro:thruster_joint name="surge_port_hi" p="${chassis_surge_port_hi}" o="${align_surge_port_hi}"/>
-  <xacro:thruster_joint name="surge_stbd_hi" p="${chassis_surge_stbd_hi}" o="${align_surge_stbd_hi}"/>
   <xacro:thruster_joint name="surge_port_lo" p="${chassis_surge_port_lo}" o="${align_surge_port_lo}"/>
   <xacro:thruster_joint name="surge_stbd_lo" p="${chassis_surge_stbd_lo}" o="${align_surge_stbd_lo}"/>

File: riptide_description/urdf/riptide_links.xacro (robot description, xacro)
@@ -175,6 +175,4 @@
     </link>
   </xacro:macro>
-  <xacro:thruster_link thruster="surge_port_hi" />
-  <xacro:thruster_link thruster="surge_stbd_hi" />
   <xacro:thruster_link thruster="surge_port_lo" />
   <xacro:thruster_link thruster="surge_stbd_lo" />

File: riptide_description/urdf/riptide_properties.xacro (robot description, xacro)
@@ -16,6 +16,4 @@
   <xacro:property name="chassis_port_battery" value="-0.1781 0.1302 -0.0140" />
   <xacro:property name="chassis_stbd_battery" value="-0.1781 -0.1302 -0.0140" />
-  <xacro:property name="chassis_surge_port_hi" value="-0.2238 0.1824 0.1384" />
-  <xacro:property name="chassis_surge_stbd_hi" value="-0.2238 -0.1824 0.1384" />
   <xacro:property name="chassis_surge_port_lo" value="-0.2238 0.1824 -0.0838" />
   <xacro:property name="chassis_surge_stbd_lo" value="-0.2238 -0.1824 -0.0838" />
@@ -68,6 +66,4 @@
   <xacro:property name="stbd_battery_mesh" value="package://riptide_description/meshes/stbd_battery.stl" />
   <xacro:property name="thruster_mesh" value="package://riptide_description/meshes/thruster.stl" />
-  <xacro:property name="align_surge_port_hi" value="0 ${-M_PI/2} ${M_PI}" />
-  <xacro:property name="align_surge_stbd_hi" value="0 ${M_PI/2} 0" />
   <xacro:property name="align_surge_port_lo" value="0 ${-M_PI/2} ${M_PI}" />
   <xacro:property name="align_surge_stbd_lo" value="0 ${M_PI/2} 0" />

File: riptide_description/urdf/riptide_simulation.xacro (robot description, xacro)
@@ -27,6 +27,4 @@
     </gazebo>
   </xacro:macro>
-  <xacro:thruster_link_gazebo name="surge_port_hi" />
-  <xacro:thruster_link_gazebo name="surge_stbd_hi" />
   <xacro:thruster_link_gazebo name="surge_port_lo" />
   <xacro:thruster_link_gazebo name="surge_stbd_lo" />
@@ -63,6 +61,4 @@
     </gazebo>
   </xacro:macro>
-  <xacro:thruster_joint_gazebo name="surge_port_hi" />
-  <xacro:thruster_joint_gazebo name="surge_stbd_hi" />
   <xacro:thruster_joint_gazebo name="surge_port_lo" />
   <xacro:thruster_joint_gazebo name="surge_stbd_lo" />
